File: Node#1/Node#1.sch (EAGLE design)
At the start: 110 parts, among them U1 BLUENRG-232, U2 SEMTECH_SX1503I091TRTSEMTECH_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, U3 MIC4468YWM, U4 LM339ADR, X1 2081-1228, X2 2081-1228, X3 2081-1228, Y1 ECS-160-12-36-AGN-TR, Y2 NX2012SA-32.768K-STD-MUB-1

Commit message: Update LBR
Connections:
- removed net N$83: X3.P2, X3.P4, X3.P6, X3.P8
- new net AGND: U$1.S, U$2.S, U$7.S, U$8.S, U3.GND
- new net V+: U3.VS, X3.P2, X3.P4, X3.P6, X3.P8
- net GND: no longer U$1.S, U$2.S, U$7.S, U$8.S, U3.GND
Other:
- moved on the sheet: X3
Changed lines of the file:
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@@
 <setting verticaltext="up"/>
 </settings>
-<grid distance="0.05" unitdist="inch" unit="inch" style="lines" multiple="1" display="no" altdistance="0.01" altunitdist="inch" altunit="inch"/>
+<grid distance="0.1" unitdist="inch" unit="inch" style="lines" multiple="1" display="no" altdistance="0.01" altunitdist="inch" altunit="inch"/>
 <layers>
 <layer number="1" name="Top" color="4" fill="1" visible="no" active="no"/>
@@
 <part name="X2" library="BlueHome" deviceset="2081-1228" device=""/>
 <part name="U3" library="BlueHome" deviceset="MIC4468YWM" device=""/>
-<part name="GND41" library="supply1" deviceset="GND" device=""/>
 <part name="U$2" library="BlueHome" deviceset="BUK9840-55" device=""/>
 <part name="R39" library="rcl" deviceset="R-EU_" device="R1210"/>
@@
 <part name="R42" library="rcl" deviceset="R-EU_" device="R1210"/>
 <part name="U$8" library="BlueHome" deviceset="BUK9840-55" device=""/>
-<part name="GND42" library="supply1" deviceset="GND" device=""/>
 <part name="U4" library="BlueHome" deviceset="LM339ADR" device=""/>
+<part name="P+2" library="supply1" deviceset="V+" device=""/>
+<part name="AGND1" library="supply1" deviceset="AGND" device=""/>
+<part name="AGND2" library="supply1" deviceset="AGND" device=""/>
 </parts>
 <sheets>
@@
 <instance part="GND27" gate="1" x="307.34" y="101.6" rot="R180"/>
 <instance part="GND28" gate="1" x="302.26" y="91.44" rot="R90"/>
-<instance part="X3" gate="G$1" x="279.4" y="15.24" rot="R90"/>
+<instance part="X3" gate="G$1" x="279.4" y="35.56" rot="R90"/>
 <instance part="LED2" gate="G$1" x="330.2" y="90.17"/>
 <instance part="D6" gate="G$1" x="337.82" y="92.71" rot="R270"/>
@@
 <instance part="X2" gate="G$1" x="278.13" y="-59.69" rot="R90"/>
 <instance part="U3" gate="G$1" x="142.24" y="-20.32"/>
-<instance part="GND41" gate="1" x="175.26" y="-35.56"/>
 <instance part="U$2" gate="G$1" x="266.7" y="-12.7"/>
 <instance part="R39" gate="G$1" x="236.22" y="-10.16"/>
@@
 <instance part="R42" gate="G$1" x="297.18" y="-25.4"/>
 <instance part="U$8" gate="G$1" x="307.34" y="-22.86"/>
-<instance part="GND42" gate="1" x="279.4" y="-39.37"/>
 <instance part="U4" gate="A" x="374.65" y="-19.05"/>
+<instance part="P+2" gate="1" x="210.82" y="17.78"/>
+<instance part="AGND1" gate="VR1" x="175.26" y="-35.56"/>
+<instance part="AGND2" gate="VR1" x="279.4" y="-40.64"/>
 </instances>
 <busses>
@@
 <pinref part="GND40" gate="1" pin="GND"/>
 </segment>
-<segment>
-<pinref part="U3" gate="G$1" pin="GND"/>
-<pinref part="GND41" gate="1" pin="GND"/>
-<wire x1="165.1" y1="-30.48" x2="175.26" y2="-30.48" width="0.1524" layer="91"/>
-<wire x1="175.26" y1="-30.48" x2="175.26" y2="-33.02" width="0.1524" layer="91"/>
-</segment>
-<segment>
-<pinref part="U$1" gate="G$1" pin="S"/>
-<wire x1="248.92" y1="-12.7" x2="248.92" y2="-31.75" width="0.1524" layer="91"/>
-<pinref part="U$8" gate="G$1" pin="S"/>
-<wire x1="248.92" y1="-31.75" x2="269.24" y2="-31.75" width="0.1524" layer="91"/>
-<wire x1="269.24" y1="-31.75" x2="279.4" y2="-31.75" width="0.1524" layer="91"/>
-<wire x1="279.4" y1="-31.75" x2="289.56" y2="-31.75" width="0.1524" layer="91"/>
-<wire x1="289.56" y1="-31.75" x2="309.88" y2="-31.75" width="0.1524" layer="91"/>
-<wire x1="309.88" y1="-31.75" x2="309.88" y2="-27.94" width="0.1524" layer="91"/>
-<pinref part="U$7" gate="G$1" pin="S"/>
-<wire x1="289.56" y1="-22.86" x2="289.56" y2="-31.75" width="0.1524" layer="91"/>
-<junction x="289.56" y="-31.75"/>
-<pinref part="U$2" gate="G$1" pin="S"/>
-<wire x1="269.24" y1="-17.78" x2="269.24" y2="-31.75" width="0.1524" layer="91"/>
-<junction x="269.24" y="-31.75"/>
-<wire x1="279.4" y1="-31.75" x2="279.4" y2="-36.83" width="0.1524" layer="91"/>
-<junction x="279.4" y="-31.75"/>
-<pinref part="GND42" gate="1" pin="GND"/>
-</segment>
 </net>
 <net name="N$15" class="0">
@@
 <pinref part="X3" gate="G$1" pin="P7"/>
 <wire x1="248.92" y1="6.35" x2="266.7" y2="6.35" width="0.1524" layer="91"/>
-<wire x1="266.7" y1="6.35" x2="266.7" y2="13.97" width="0.1524" layer="91"/>
+<wire x1="266.7" y1="6.35" x2="266.7" y2="34.29" width="0.1524" layer="91"/>
 </segment>
 </net>
@@
 <pinref part="X3" gate="G$1" pin="P1"/>
 <wire x1="309.88" y1="6.35" x2="297.18" y2="6.35" width="0.1524" layer="91"/>
-<wire x1="297.18" y1="6.35" x2="297.18" y2="13.97" width="0.1524" layer="91"/>
+<wire x1="297.18" y1="6.35" x2="297.18" y2="34.29" width="0.1524" layer="91"/>
 </segment>
 </net>
@@
 <pinref part="X3" gate="G$1" pin="P3"/>
 <wire x1="289.56" y1="6.35" x2="287.02" y2="6.35" width="0.1524" layer="91"/>
-<wire x1="287.02" y1="6.35" x2="287.02" y2="13.97" width="0.1524" layer="91"/>
+<wire x1="287.02" y1="6.35" x2="287.02" y2="34.29" width="0.1524" layer="91"/>
 </segment>
 </net>
@@
 <pinref part="X3" gate="G$1" pin="P5"/>
 <wire x1="269.24" y1="6.35" x2="276.86" y2="6.35" width="0.1524" layer="91"/>
-<wire x1="276.86" y1="6.35" x2="276.86" y2="13.97" width="0.1524" layer="91"/>
-</segment>
-</net>
-<net name="N$83" class="0">
+<wire x1="276.86" y1="6.35" x2="276.86" y2="34.29" width="0.1524" layer="91"/>
+</segment>
+</net>
+<net name="V+" class="0">
 <segment>
 <pinref part="X3" gate="G$1" pin="P2"/>
-<wire x1="292.1" y1="13.97" x2="292.1" y2="8.89" width="0.1524" layer="91"/>
-<wire x1="292.1" y1="8.89" x2="281.94" y2="8.89" width="0.1524" layer="91"/>
-<wire x1="281.94" y1="8.89" x2="271.78" y2="8.89" width="0.1524" layer="91"/>
-<wire x1="271.78" y1="8.89" x2="261.62" y2="8.89" width="0.1524" layer="91"/>
-<wire x1="261.62" y1="8.89" x2="248.92" y2="8.89" width="0.1524" layer="91"/>
-<wire x1="248.92" y1="8.89" x2="248.92" y2="20.32" width="0.1524" layer="91"/>
+<wire x1="292.1" y1="34.29" x2="292.1" y2="10.16" width="0.1524" layer="91"/>
+<wire x1="292.1" y1="10.16" x2="281.94" y2="10.16" width="0.1524" layer="91"/>
+<wire x1="281.94" y1="10.16" x2="271.78" y2="10.16" width="0.1524" layer="91"/>
+<wire x1="271.78" y1="10.16" x2="261.62" y2="10.16" width="0.1524" layer="91"/>
 <pinref part="X3" gate="G$1" pin="P8"/>
-<wire x1="261.62" y1="13.97" x2="261.62" y2="8.89" width="0.1524" layer="91"/>
-<junction x="261.62" y="8.89"/>
+<wire x1="261.62" y1="34.29" x2="261.62" y2="10.16" width="0.1524" layer="91"/>
+<junction x="261.62" y="10.16"/>
 <pinref part="X3" gate="G$1" pin="P6"/>
-<wire x1="271.78" y1="13.97" x2="271.78" y2="8.89" width="0.1524" layer="91"/>
-<junction x="271.78" y="8.89"/>
+<wire x1="271.78" y1="34.29" x2="271.78" y2="10.16" width="0.1524" layer="91"/>
+<junction x="271.78" y="10.16"/>
 <pinref part="X3" gate="G$1" pin="P4"/>
-<wire x1="281.94" y1="13.97" x2="281.94" y2="8.89" width="0.1524" layer="91"/>
-<junction x="281.94" y="8.89"/>
-</segment>
-</net>
+<wire x1="281.94" y1="34.29" x2="281.94" y2="10.16" width="0.1524" layer="91"/>
+<junction x="281.94" y="10.16"/>
+<pinref part="U3" gate="G$1" pin="VS"/>
+<wire x1="165.1" y1="-25.4" x2="210.82" y2="-25.4" width="0.1524" layer="91"/>
+<wire x1="210.82" y1="-25.4" x2="210.82" y2="10.16" width="0.1524" layer="91"/>
+<wire x1="210.82" y1="10.16" x2="261.62" y2="10.16" width="0.1524" layer="91"/>
+<wire x1="210.82" y1="10.16" x2="210.82" y2="15.24" width="0.1524" layer="91"/>
+<junction x="210.82" y="10.16"/>
+<pinref part="P+2" gate="1" pin="V+"/>
+</segment>
+</net>
+<net name="AGND" class="0">
+<segment>
+<pinref part="U3" gate="G$1" pin="GND"/>
+<wire x1="165.1" y1="-30.48" x2="175.26" y2="-30.48" width="0.1524" layer="91"/>
+<wire x1="175.26" y1="-30.48" x2="175.26" y2="-33.02" width="0.1524" layer="91"/>
+<pinref part="AGND1" gate="VR1" pin="AGND"/>
+</segment>
+<segment>
+<pinref part="U$1" gate="G$1" pin="S"/>
+<wire x1="248.92" y1="-12.7" x2="248.92" y2="-31.75" width="0.1524" layer="91"/>
+<pinref part="U$8" gate="G$1" pin="S"/>
+<wire x1="248.92" y1="-31.75" x2="269.24" y2="-31.75" width="0.1524" layer="91"/>
+<wire x1="269.24" y1="-31.75" x2="279.4" y2="-31.75" width="0.1524" layer="91"/>
+<wire x1="279.4" y1="-31.75" x2="289.56" y2="-31.75" width="0.1524" layer="91"/>
+<wire x1="289.56" y1="-31.75" x2="309.88" y2="-31.75" width="0.1524" layer="91"/>
+<wire x1="309.88" y1="-31.75" x2="309.88" y2="-27.94" width="0.1524" layer="91"/>
+<pinref part="U$7" gate="G$1" pin="S"/>
+<wire x1="289.56" y1="-22.86" x2="289.56" y2="-31.75" width="0.1524" layer="91"/>
+<junction x="289.56" y="-31.75"/>
+<pinref part="U$2" gate="G$1" pin="S"/>
+<wire x1="269.24" y1="-17.78" x2="269.24" y2="-31.75" width="0.1524" layer="91"/>
+<junction x="269.24" y="-31.75"/>
+<wire x1="279.4" y1="-31.75" x2="279.4" y2="-35.56" width="0.1524" layer="91"/>
+<junction x="279.4" y="-31.75"/>
+<pinref part="AGND2" gate="VR1" pin="AGND"/>
+<wire x1="279.4" y1="-35.56" x2="279.4" y2="-36.83" width="0.1524" layer="91"/>
+<wire x1="279.4" y1="-36.83" x2="279.4" y2="-38.1" width="0.1524" layer="91"/>
+</segment>
+</net>

Commit message: Update Endstufe Absicherung
Parts:
- added C18, C19, C20, C21, C22, C23: (no value), rcl:C-EUC0805
- added C24, C25: (no value), rcl:CPOL-EUSMCC
- added LED17: (no value), led:LED3MM
- added R43, R44, R45, R46, R47, R48, R49, R50, R51: (no value), rcl:R-EU_R1210
- added U5: 74HC08D,652, BlueHome:74HC08D,652
- added U6: SN74LVC1G74DCUR, BlueHome:SN74LVC1G74DCUR
- added U7: TMP75BID, BlueHome:TMP75BID
- added U8: IRM-05-5, BlueHome:IRM-05-5
- added U9: LMS8117AMP-3.3, BlueHome:LMS8117AMP-3.3
- added VR1: TS53YJ103MR10, BlueHome:TS53YJ103MR10
Connections:
- new net ERROR: R49.1, U3.1B, U3.2B, U3.3B, U3.4B, U5.4Y
- new net E_RESET: U6.CLK
- new net N$100: X3.P2, X3.P4, X3.P6, X3.P8
- new net N$82: R43.1, VR1.C
- new net N$83: R43.2, R44.1, U4.1IN+, U4.2IN+, U4.3IN+, U4.4IN+
- new net N$84: R45.2, U4.1IN-
- new net N$85: U4.1OUT, U5.1A
- new net N$86: R48.2, U4.4IN-
- new net N$87: R47.2, U4.3IN-
- new net N$88: R46.2, U4.2IN-
- new net N$89: U4.2OUT, U5.1B
- new net N$90: U4.OUT4, U5.2A
- new net N$91: U4.OUT3, U5.2B
- new net N$92: U5.1Y, U5.3A
- new net N$93: U5.2Y, U5.3B
- new net N$94: U5.3Y, U6.~CLR
- new net N$95: U8.AC(L)
- new net N$96: U5.4B, U6.Q
- new net N$97: R50.1, U5.4A, U7.ALERT
- new net N$98: U8.AC(N)
- net +3V3: now also C18.2, C19.1, C20.2, C21.2, C23.1, C25.+, LED17.A, R50.2, U4.VCC, U5.VCC, U6.D, U6.VCC, U6.~PRE, U7.V+, U9.OUT, U9.VOUT
- net +5V: now also C22.1, C24.+, U8.+V, U9.IN
- net AGND: now also R51.1, VR1.A, VR1.B
- net GND: now also C18.1, C19.2, C20.1, C21.1, C22.2, C23.2, C24.-, C25.-, R51.2, U4.GND, U5.GND, U6.GND, U7.A0, U7.A1, U7.A2, U7.GND, U8.-V, U9.GND, X2.P1, X2.P2, X2.P3, X2.P4, X2.P5, X2.P6, X2.P7, X2.P8
- net N$44: now also LED17.C, R49.2; no longer U3.1B, U3.2B, U3.3B, U3.4B
- net N$78: now also R45.1
- net N$79: now also R48.1
- net N$80: now also R47.1
- net N$81: now also R46.1
- net SCL: now also U7.SCL
- net SDA: now also U7.SDA
- net V+: now also R44.2; no longer X3.P2, X3.P4, X3.P6, X3.P8
Other:
- note added: "PLACEHOLDER STAR GROUNDING"
- moved on the sheet: U4, X1, X2

Commit message: Node#1 update
Parts:
- added C26, C27: (no value), rcl:C-EUC0805
- added J1: 1757242, BlueHome:1757242
- added J2: DCJ200-10-A-XX-X_REVA, BlueHome:DCJ200-10-A-XX-X_REVA
- added JMP2, JMP3, JMP4, JMP5, JMP6: 0R-JUMPA, jump-0r-smd:0R-JUMPA
- added K1, K2, K3, K4: FTR-K1CK005W, BlueHome:FTR-K1CK005W
- added R52, R54, R55: (no value), rcl:R-EU_R0805
- added R53: (no value), rcl:R-EU_R1210
- added U$9: RND170-00004, BlueHome:RND170-00004
- added U10: ULN2003AIDG4, BlueHome:ULN2003AIDG4
- added X4: 2081-1222, BlueHome:2081-1222
Connections:
- new net N$101: JMP3-0R.1, U10.2B
- new net N$102: JMP4-0R.1, U10.3B
- new net N$103: JMP5-0R.1, U10.4B
- new net N$104: J1.2, U$9.P$1
- new net N$105: C26.2, JMP6-0R.2, U3.VS
- new net N$106: K1.COIL_1, U10.1C
- new net N$107: J2.3, R53.1
- new net N$108: K2.COIL_1, U10.2C
- new net N$109: K3.COIL_1, U10.3C
- new net N$110: K4.COIL_1, U10.4C
- new net N$111: R54.1, X3.P8
- new net N$114: K1.NO_2
- new net N$115: K1.COM_2
- new net N$116: K2.COM_2
- new net N$117: K3.COM_2
- new net N$118: K4.COM_2
- new net N$119: K1.COM_1
- new net N$120: K2.COM_1
- new net N$121: K3.COM_1
- new net N$122: K4.COM_1
- new net N$123: K2.NO_2
- new net N$124: K3.NO_2
- new net N$125: K4.NO_2
- new net N$99: JMP2-0R.1, U10.1B
- net +3V3: now also R52.2, R53.2
- net +5V: now also C27.2, JMP6-0R.3, K1.COIL_2, K2.COIL_2, K3.COIL_2, K4.COIL_2, U10.E
- net AGND: now also C26.1, C27.1, J2.2, U10.COM, X4.P2
- net DIO2: now also JMP2-0R.2
- net DIO3: now also JMP3-0R.2
- net DIO6: now also JMP4-0R.2
- net DIO7: now also JMP5-0R.2
- net ERROR: now also R52.1
- net N$100: now also R54.2; no longer X3.P8
- net N$39: now also JMP5-0R.3
- net N$55: now also JMP2-0R.3
- net N$56: now also JMP3-0R.3
- net N$57: now also JMP4-0R.3
- net N$95: now also U$9.P$2
- net N$98: now also J1.1
- net V+: now also J2.1, JMP6-0R.1, X4.P1; no longer U3.VS
Other:
- note added: "DC-DC"
- note added: "RELAIS"
- moved on the sheet: C22, C23, C24, C25, R51, U8, U9

Commit message: Node#1
Parts:
- removed D2, D3, D4, D5, D6, D7, D8, D9: BAS40-06, diode:BAS40-06
- added C28, C29, C30, C31, C32, C33: (no value), rcl:C-EUC0805
- added JP6: (no value), pinhead:PINHD-1X2
- added R56, R57, R58, R59, R60, R61, R62, R63, R64, R65, R66, R67: (no value), rcl:R-EU_R1210
- added S2: FSM4JSMAATR, BlueHome:FSM4JSMAATR
- added U$10, U$11, U$12, U$13, U$14, U$15, U$16, U$17, U$18, U$19: BZB984, BlueHome:BZB984
- added U11, U12: ACS723LLCTR-40AB-T, BlueHome:ACS723LLCTR-40AB-T
- R54, R55: device rcl:R-EU_R0805 -> rcl:R-EU_R1210
Connections:
- removed net N$107: J2.3, R53.1
- removed net N$115: K1.COM_2
- removed net N$116: K2.COM_2
- removed net N$117: K3.COM_2
- removed net N$118: K4.COM_2
- removed net N$119: K1.COM_1
- removed net N$120: K2.COM_1
- removed net N$121: K3.COM_1
- removed net N$122: K4.COM_1
- removed net N$123: K2.NO_2
- removed net N$124: K3.NO_2
- removed net N$125: K4.NO_2
- removed net N$45: JP7.1, R16.1
- removed net N$96: U5.4B, U6.Q
- removed net N$97: R50.1, U5.4A, U7.ALERT
- new net JACK: J2.3, R16.1, R53.1
- new net L1: K1.NO_1, K1.NO_2, R48.1, U$8.D, X3.P1
- new net L2: K1.COM_1, R57.2, U12.IP-, X3.P2
- new net L3: K2.NO_1, K2.NO_2, R47.1, U$7.D, X3.P3
- new net L4: K2.COM_1, K2.COM_2, R56.2, X3.P4
- new net L5: K3.NO_1, K3.NO_2, R46.1, U$2.D, X3.P5
- new net L6: K3.COM_1, K3.COM_2, R54.2, X3.P6
- new net L7: K4.NO_1, K4.NO_2, R45.1, U$1.D, X3.P7
- new net L8: K4.COM_1, K4.COM_2, R55.2, X3.P8
- new net N$112: K1.COM_2, U12.IP+
- new net N$113: R63.2, U11.VIOUT
- net +3V3: now also C32.1, R66.2
- net +5V: now also C28.1, C29.2, U11.VCC, U12.VCC
- net ADC1: now also R63.1, R64.2, U$18.2
- net ADC2: now also R62.2, R65.2, U$19.1
- net DIO12: now also U5.4B, U6.Q
- net DIO13: now also R50.1, U5.4A, U7.ALERT
- net DIO14: now also C30.1, JP6.1, R66.1, S2.1, S2.2
- net GND: now also C28.2, C29.1, C30.2, C31.2, C32.2, C33.2, JP7.1, R64.1, R65.1, R67.1, U$10.3, U$11.3, U$12.3, U$13.3, U$14.3, U$15.3, U$16.3, U$17.3, U$18.3, U$19.3, U11.BW_SEL, U11.GND, U12.BW_SEL, U12.GND; no longer D2.AA, D3.AA, D4.AA, D5.AA, D6.AA, D7.AA, D8.AA, D9.AA
- net N$100: now also R54.1, R55.1, R56.1, R57.1, U11.IP-; no longer R54.2, X3.P2, X3.P4, X3.P6
- net N$106: now also R58.1; no longer K1.COIL_1
- net N$108: now also R59.1; no longer K2.COIL_1
- net N$109: now also R60.1; no longer K3.COIL_1
- net N$110: now also R61.1; no longer K4.COIL_1
- net N$111: now also R62.1, U12.VIOUT; no longer R54.1, X3.P8
- net N$114: now also JP6.2, R67.2, S2.3, S2.4; no longer K1.NO_2
- net N$12: now also C33.1
- net N$13: now also C31.1
- net N$15: now also U$13.1; no longer D2.K1
- net N$20: now also U$12.2; no longer D3.K2
- net N$21: now also U$11.1; no longer D4.K1
- net N$22: now also U$11.2; no longer D4.K2
- net N$23: now also U$14.2; no longer D6.K2
- net N$25: now also U$14.1; no longer D6.K1
- net N$27: now also U$15.1; no longer D7.K1
- net N$28: now also U$15.2; no longer D7.K2
- net N$29: now also U$16.1; no longer D8.K1
- net N$30: now also U$16.2; no longer D8.K2
- net N$31: now also U$17.1; no longer D9.K1
- net N$32: now also U$17.2; no longer D9.K2
- net N$35: now also U$13.2; no longer D2.K2
- net N$37: now also U$12.1; no longer D3.K1
- net N$47: now also U$10.1; no longer D5.K1
- net N$50: now also U$10.2; no longer D5.K2
- net N$78: now also K1.COIL_1, R58.2; no longer R45.1, U$1.D, X3.P7
- net N$79: now also K2.COIL_1, R59.2; no longer R48.1, U$8.D, X3.P1
- net N$80: now also K3.COIL_1, R60.2; no longer R47.1, U$7.D, X3.P3
- net N$81: now also K4.COIL_1, R61.2; no longer R46.1, U$2.D, X3.P5
- net V+: now also U11.IP+
Other:
- moved on the sheet: JP3, JP5, R54, R55
