File: Node#1/Node#1.sch (EAGLE design)
At the start: 187 parts, among them J1 1757242, J2 DCJ200-10-A-XX-X_REVA, K1 FTR-K1CK005W, K2 FTR-K1CK005W, K3 FTR-K1CK005W, K4 FTR-K1CK005W, U1 BLUENRG-232, U10 ULN2003AIDG4, U11 ACS723LLCTR-40AB-T, U12 ACS723LLCTR-40AB-T, U2 SEMTECH_SX1503I091TRTSEMTECH_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, U3 MIC4468YWM, U4 LM339ADR, U5 74HC08D,652, U6 SN74LVC1G74DCUR, U7 TMP75BID, U8 IRM-05-5, U9 LMS8117AMP-3.3, X1 2081-1228, X2 2081-1228, X3 2081-1228, X4 2081-1222, Y1 ECS-160-12-36-AGN-TR, Y2 NX2012SA-32.768K-STD-MUB-1

Commit message: Node#2 sorted, Node#1 small adjusts
Parts:
- removed C28: (no value), rcl:C-EUC0805
- removed R63, R64: (no value), rcl:R-EU_R1210
- removed U$18: BZB984, BlueHome:BZB984
- removed U11: ACS723LLCTR-40AB-T, BlueHome:ACS723LLCTR-40AB-T
- added C39: 1u, rcl:C-EUC0805
- added C40: 100n, rcl:C-EUC0805
- added C41: 100mF, rcl:C-EU050-055X075
- added C42: (no value), rcl:C-EUC0805
- added D3: MUR150RL, diode:MUR150RL
- added R5: (no value), rcl:R-EU_R0805
- added R6, R70: (no value), rcl:R-EU_R1210
- added U$22, U$6: BZB984, BlueHome:BZB984
- added U13: RV8564C3, BlueHome:RV8564C3
- added U14: ACS723LLCTR-40AB-T, BlueHome:ACS723LLCTR-40AB-T
- C38: device rcl:C-EUC0805 -> rcl:CPOL-EU150CLZ-1010
Connections:
- net N$101 renamed RELAY2
- net N$102 renamed RELAY3
- net N$103 renamed RELAY4
- net N$99 renamed RELAY1
- removed net N$100: R54.1, R55.1, R56.1, R57.1, U11.IP-
- removed net N$112: K1.COM_2, U12.IP+
- removed net N$113: R63.2, U11.VIOUT
- new net +3V3_RTC: C39.2, C40.2, C41.1, D3.C, U$6.2, U13.VDD
- new net CURR_SENS_PWM: R54.1, R55.1, R56.1, R57.1, U14.IP-
- new net CURR_SENS_RELAY: K1.COM_1, K1.COM_2, U12.IP+
- new net N$8: D3.A, R5.1
- new net N$96: R6.1, U14.VIOUT
- net +5V: now also C42.2, R5.2, U14.VCC; no longer C28.1, U11.VCC
- net ADC1: no longer R63.1, R64.2, U$18.2
- net ADC2: now also R6.2, R70.2, U$22.1
- net AGND: now also C38.-; no longer C38.2
- net DIO12: now also U13.INT
- net GND: now also C39.1, C40.1, C41.2, C42.1, R70.1, U$22.3, U$6.3, U13.CLKOE, U13.GND, U14.BW_SEL, U14.GND; no longer C28.2, R64.1, U$18.3, U11.BW_SEL, U11.GND
- net L1: now also R45.1, U$8.D2; no longer R48.1
- net L2: no longer K1.COM_1
- net L3: now also R46.1, U$7.D2; no longer R47.1
- net L5: now also R47.1, U$2.D2; no longer R46.1
- net L7: now also R48.1, U$1.D2; no longer R45.1
- net N$116: no longer C38.1
- net SCL: now also U13.SCL
- net SDA: now also U13.SDA
- net V+: now also C38.+, U14.IP+; no longer U11.IP+
Other:
- note added: "BlueNRG2 Processor"
- note added: "Current Sensing"
- note added: "Jumper"
- note added: "MOSFET Option"
- note added: "Port Expander"
- note added: "Power Supply"
- note added: "Relay Option"

Commit message: Schematic finished (hopefully) !
Parts:
- removed L1: (no value), rcl:L-EUL5650M
- added U$18: LIND, BlueHome:LIND
- U$3, U$4: value L -> L0402; device BlueHome:L -> BlueHome:L0402
Connections:
- net N$15 renamed IO0
- net N$20 renamed IO3
- net N$21 renamed IO4
- net N$22 renamed IO5
- net N$23 renamed IO9
- net N$25 renamed IO8
- net N$27 renamed IO10
- net N$28 renamed IO11
- net N$29 renamed IO12
- net N$30 renamed IO13
- net N$31 renamed IO14
- net N$32 renamed IO15
- net N$35 renamed IO1
- net N$37 renamed IO2
- net N$47 renamed IO6
- net N$50 renamed IO7
- removed net N$18: R9.1, X1.P7
- removed net N$24: R13.1, X1.P5
- removed net N$26: R24.1, X1.P4
- removed net N$34: R25.1, X1.P3
- removed net N$36: R8.1, X1.P8
- removed net N$40: R12.1, X1.P6
- removed net N$48: JP7.2, R21.1
- removed net N$59: R29.1, X1.P1
- removed net N$61: R28.1, X1.P2
- removed net N$63: JP7.4, R33.1
- removed net N$65: JP7.3, R32.1
- removed net N$68: JP7.6, R37.1
- removed net N$71: JP7.5, R36.1
- new net O_IO0: R8.1, X1.P1
- new net O_IO1: R9.1, X1.P2
- new net O_IO10: R28.1
- new net O_IO11: JP7.2, R29.1, R32.1
- new net O_IO12: JP7.3, R33.1
- new net O_IO13: JP7.4, R36.1
- new net O_IO14: JP7.5, R37.1
- new net O_IO15: JP7.6
- new net O_IO2: R12.1, X1.P3
- new net O_IO3: R13.1, X1.P4
- new net O_IO4: R16.1, X1.P5
- new net O_IO5: R17.1, X1.P6
- new net O_IO6: R20.1, X1.P7
- new net O_IO7: R21.1, X1.P8
- new net O_IO8: R24.1
- new net O_IO9: R25.1
- net E_SHORT: no longer R17.1
- net E_TEMP: no longer R20.1
- net JACK: no longer R16.1
- net N$107: now also U$18.1; no longer L1.1
- net N$116: now also U$18.2; no longer L1.2
Other:
- note added: "MOSFET Error Detection"
- moved on the sheet: C31, C32, C33, JP3, JP5, JP7, LED1, LED10, LED11, LED12, LED13, LED14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

Commit message: Changed Packages, connected GPIO
Parts:
- added R63: (no value), rcl:R-EU_R0805
- added U$23: STAR_GROUND, BlueHome:STAR_GROUND
- R51: device rcl:R-EU_R1210 -> rcl:R-EU_R0805
Connections:
- new net DIO0: R51.1
- new net DIO1: R63.1
- net AGND: now also U$23.P$1; no longer R51.1
- net GND: now also U$23.P$2; no longer R51.2
- net TDI: now also R51.2
- net TDO: now also R63.2

Commit message: Created BlueNRG Design Block and Board Size for Node#1
Parts:
- removed ANT1: CONUFL001-SMD, BlueHome:CONUFL001-SMD
- removed C1, C10, C3, C5, C8: (no value), rcl:C-EUC0805K
- removed C11, C12, C13, C14, C15, C30: (no value), rcl:C-EUC0805
- removed C16, C17: (no value), rcl:C-EUC0402
- removed D1: BAS40-06, diode:BAS40-06
- removed JMP1: 0R-JUMPA, jump-0r-smd:0R-JUMPA
- removed JP1: (no value), pinhead:PINHD-2X5
- removed JP2: (no value), jumper:JP1E
- removed JP4: (no value), pinhead:PINHD-1X3
- removed JP6: (no value), pinhead:PINHD-1X2
- removed R1, R2, R3, R4, R51, R63: (no value), rcl:R-EU_R0805
- removed R66, R67: (no value), rcl:R-EU_R1210
- removed S1, S2: FSM4JSMAATR, BlueHome:FSM4JSMAATR
- removed U$3, U$4: L0402, BlueHome:L0402
- removed U$5: BALF-NRG-01D3, BlueHome:BALF-NRG-01D3
- removed U1: BLUENRG-232, BlueHome:BLUENRG-232
- removed Y1: ECS-160-12-36-AGN-TR, BlueHome:ECS-160-12-36-AGN-TR
- removed Y2: NX2012SA-32.768K-STD-MUB-1, BlueHome:NX2012SA-32.768K-STD-MUB-1
- added ANT2: CONUFL001-SMD, BlueHome:CONUFL001-SMD
- added C43, C45, C47, C48, C50: (no value), rcl:C-EUC0805K
- added C52, C53, C54, C55, C56, C57: (no value), rcl:C-EUC0805
- added C58, C59: (no value), rcl:C-EUC0402
- added D4: BAS40-06, diode:BAS40-06
- added JMP7: 0R-JUMPA, jump-0r-smd:0R-JUMPA
- added JP10: (no value), jumper:JP1E
- added JP11: (no value), pinhead:PINHD-1X3
- added JP12: (no value), pinhead:PINHD-1X2
- added JP9: (no value), pinhead:PINHD-2X5
- added R64, R71, R72, R73, R76, R77: (no value), rcl:R-EU_R0805
- added R74, R75: (no value), rcl:R-EU_R1210
- added S3, S4: FSM4JSMAATR, BlueHome:FSM4JSMAATR
- added U$24, U$26: L0402, BlueHome:L0402
- added U$25: BALF-NRG-01D3, BlueHome:BALF-NRG-01D3
- added U11: BLUENRG-232, BlueHome:BLUENRG-232
- added Y3: ECS-160-12-36-AGN-TR, BlueHome:ECS-160-12-36-AGN-TR
- added Y4: NX2012SA-32.768K-STD-MUB-1, BlueHome:NX2012SA-32.768K-STD-MUB-1
- renumbered C2 to C28, C4 to C44, C6 to C46, C7 to C49, C9 to C51
Connections:
- removed net 0V: C12.2, C13.1
- removed net N$1: C49.1, C8.1, U1.VDD1V2
- removed net N$10: C14.1, U1.SXTAL0, Y2.2
- removed net N$11: C15.1, U1.SXTAL1, Y2.1
- removed net N$114: JP6.2, R67.2, S2.3, S2.4
- removed net N$14: U$5.RX_N, U1.RF1
- removed net N$16: C17.1, U$3.1, U$5.ANT
- removed net N$17: ANT1.SIG, C16.1, U$3.2
- removed net N$2: C10.1, C51.1, JMP1-0R.2, U1.SMPSFILT1
- removed net N$3: JP1.1, JP2.1
- removed net N$4: C12.1, U1.FXTAL1, Y1.OUT/IN
- removed net N$5: R2.1, S1.1, S1.2
- removed net N$6: C13.2, U1.FXTAL0, Y1.IN/OUT
- removed net N$7: U$5.RX_P, U1.RF0
- removed net N$9: C14.2, C15.2, U$4.1
- new net N$15: C48.1, C49.1, U11.VDD1V2
- new net N$18: C50.1, C51.1, JMP7-0R.2, U11.SMPSFILT1
- new net N$20: R71.1, S3.1, S3.2
- new net N$21: C53.1, U11.FXTAL1, Y3.OUT/IN
- new net N$22: C54.2, U11.FXTAL0, Y3.IN/OUT
- new net N$23: C55.2, C56.2, U$24.1
- new net N$24: C55.1, U11.SXTAL0, Y4.2
- new net N$25: C56.1, U11.SXTAL1, Y4.1
- new net N$26: C58.1, U$25.ANT, U$26.1
- new net N$27: ANT2.SIG, C59.1, U$26.2
- new net N$28: JP10.1, JP9.1
- new net N$29: JP12.2, R75.2, S4.3, S4.4
- new net N$30: U$25.RX_P, U11.RF1
- new net N$31: U$25.RX_N, U11.RF0
- net +3V3: now also C43.1, C45.1, C47.1, D4.K2, JMP7-0R.3, JP10.2, R64.2, R72.2, R73.2, R74.2, U11.VBAT1, U11.VBAT2, U11.VBAT3; no longer C1.1, C3.1, C5.1, D1.K2, JMP1-0R.3, JP2.2, R1.2, R3.2, R4.2, R66.2, U1.VBAT1, U1.VBAT2, U1.VBAT3
- net ADC1: now also U11.ADC1; no longer U1.ADC1
- net ADC2: now also U11.ADC2; no longer U1.ADC2
- net DIO0: now also R76.1; no longer R51.1
- net DIO1: now also R77.1; no longer R63.1
- net DIO12: now also U11.DIO12; no longer U1.DIO12
- net DIO13: now also U11.DIO13; no longer U1.DIO13
- net DIO14: now also C57.1, JP12.1, R74.1, S4.1, S4.2, U11.DIO14/ANATEST0; no longer C30.1, JP6.1, R66.1, S2.1, S2.2, U1.DIO14/ANATEST0
- net DIO2: now also U11.DIO2; no longer U1.DIO2
- net DIO3: now also U11.DIO3; no longer U1.DIO3
- net DIO6: now also U11.DIO6; no longer U1.DIO6
- net DIO7: now also U11.DIO7/BOOT; no longer U1.DIO7/BOOT
- net GND: now also ANT2.GND_1, ANT2.GND_2, C43.2, C45.2, C47.2, C48.2, C50.2, C52.1, C53.2, C54.1, C57.2, C58.2, C59.2, JP11.3, JP9.3, JP9.5, JP9.9, R71.2, R75.1, U$24.2, U$25.GND, U11.EXP, U11.TEST, Y3.GND; no longer ANT1.GND_1, ANT1.GND_2, C1.2, C10.2, C11.1, C16.2, C17.2, C3.2, C30.2, C5.2, C8.2, JP1.3, JP1.5, JP1.9, JP4.3, R2.2, R67.1, U$4.2, U$5.GND, U1.EXP, U1.TEST, Y1.GND
- net JTCK: now also JP9.4, U11.DIO9; no longer JP1.4, U1.DIO9
- net JTMS: now also JP9.2, U11.DIO10; no longer JP1.2, U1.DIO10
- net RESETN: now also C52.2, D4.AA, JP9.10, R64.1, S3.3, S3.4, U11.RESETN; no longer C11.2, D1.AA, JP1.10, R1.1, S1.3, S1.4, U1.RESETN
- net RXD: now also JP11.2, U11.DIO11; no longer JP4.2, U1.DIO11
- net SCL: now also R72.1, U11.DIO4; no longer R3.1, U1.DIO4
- net SDA: now also R73.1, U11.DIO5; no longer R4.1, U1.DIO5
- net SMPSFILT2: now also JMP7-0R.1, U11.SMPSFILT2; no longer JMP1-0R.1, U1.SMPSFILT2
- net TDI: now also JP9.8, R76.2, U11.DIO0; no longer JP1.8, R51.2, U1.DIO0
- net TDO: now also JP9.6, R77.2, U11.DIO1; no longer JP1.6, R63.2, U1.DIO1
- net TXD: now also JP11.1, U11.DIO8; no longer JP4.1, U1.DIO8

Commit message: Worked on Layout for Node#1
Parts:
- added X5: (no value), con-wago-500:W237-102
- R39, R40, R41, R42, R43, R44, R45, R46, R47, R48, R49, R50, R58, R59, R6, R60, R61, R70, R74, R75: device rcl:R-EU_R1210 -> rcl:R-EU_M0805
- R52: device rcl:R-EU_R0805 -> rcl:R-EU_M0805
Connections:
- net L1: now also X3.P8, X5-2.KL; no longer X3.P1
- net L2: now also X3.P7, X5-1.KL; no longer X3.P2
- net L3: now also X3.P6; no longer X3.P3
- net L4: now also X3.P5; no longer X3.P4
- net L5: now also X3.P4; no longer X3.P5
- net L6: now also X3.P3; no longer X3.P6
- net L7: now also X3.P2; no longer X3.P7
- net L8: now also X3.P1; no longer X3.P8

Commit message: Redone Node#1 Layout
Parts:
- removed LED16, LED2, LED3, LED4, LED5, LED6, LED7, LED8: (no value), led:LED3MM
- removed R23, R24, R25, R26, R27, R28, R29, R30, R31, R32, R33, R34, R35, R36, R37, R38: (no value), rcl:R-EU_R0805
- removed U$10, U$14, U$15, U$16, U$17: BZB984, BlueHome:BZB984
- added U$5: BZB984, BlueHome:BZB984
- renumbered LED1 to LED18, LED14 to LED20, LED15 to LED21, LED9 to LED19, R10 to R4, R19 to R51, R20 to R63, R21 to R66, R22 to R67, R7 to R1, R8 to R2, R9 to R3, U$12 to U$4, U$13 to U$3
Connections:
- removed net E_SHORT: U5.4B, U6.Q
- removed net E_TEMP: R50.1, U5.4A, U7.ALERT
- removed net N$54: LED2.A, R23.1
- removed net N$58: LED3.A, R26.2
- removed net N$60: LED4.A, R27.1
- removed net N$62: LED5.A, R30.2
- removed net N$64: LED6.A, R31.1
- removed net N$66: LED7.A, R34.2
- removed net N$69: LED8.A, R35.1
- removed net N$72: LED16.A, R38.2
- removed net O_IO10: R28.1
- removed net O_IO11: JP7.2, R29.1, R32.1
- removed net O_IO12: JP7.3, R33.1
- removed net O_IO13: JP7.4, R36.1
- removed net O_IO14: JP7.5, R37.1
- removed net O_IO15: JP7.6
- removed net O_IO8: R24.1
- removed net O_IO9: R25.1
- net ERROR: no longer R49.1, U5.4Y
- net GND: now also U$5.3; no longer LED16.C, LED2.C, LED3.C, LED4.C, LED5.C, LED6.C, LED7.C, LED8.C, U$10.3, U$14.3, U$15.3, U$16.3, U$17.3
- net IO10: now also R50.1, U5.4A, U7.ALERT; no longer R27.2, R28.2, U$15.1
- net IO11: now also JP7.2; no longer R29.2, R30.1, U$15.2
- net IO12: now also JP7.3; no longer R31.2, R32.2, U$16.1
- net IO13: now also JP7.4; no longer R33.2, R34.1, U$16.2
- net IO14: now also JP7.5; no longer R35.2, R36.2, U$17.1
- net IO15: now also JP7.6; no longer R37.2, R38.1, U$17.2
- net IO4: now also U$5.1; no longer U$11.1
- net IO5: now also U$5.2; no longer U$11.2
- net IO6: now also U$11.1; no longer U$10.1
- net IO7: now also U$11.2; no longer U$10.2
- net IO8: now also R49.1, U5.4Y; no longer R23.2, R24.2, U$14.1
- net IO9: now also U5.4B, U6.Q; no longer R25.2, R26.1, U$14.2
Other:
- moved on the sheet: U$11

Commit message: Arrangement of Node#1 - DC Power Jack
Parts:
- R53: device rcl:R-EU_R1210 -> rcl:R-EU_R0805
Changed lines of the file:
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@@
 <grid distance="0.1" unitdist="inch" unit="inch" style="lines" multiple="1" display="no" altdistance="0.01" altunitdist="inch" altunit="inch"/>
 <layers>
-<layer number="1" name="Top" color="4" fill="1" visible="no" active="no"/>
-<layer number="2" name="Route2" color="16" fill="1" visible="no" active="no"/>
-<layer number="3" name="Route3" color="17" fill="1" visible="no" active="no"/>
-<layer number="4" name="Route4" color="18" fill="1" visible="no" active="no"/>
-<layer number="5" name="Route5" color="19" fill="1" visible="no" active="no"/>
-<layer number="6" name="Route6" color="25" fill="1" visible="no" active="no"/>
-<layer number="7" name="Route7" color="26" fill="1" visible="no" active="no"/>
-<layer number="8" name="Route8" color="27" fill="1" visible="no" active="no"/>
-<layer number="9" name="Route9" color="28" fill="1" visible="no" active="no"/>
-<layer number="10" name="Route10" color="29" fill="1" visible="no" active="no"/>
-<layer number="11" name="Route11" color="30" fill="1" visible="no" active="no"/>
-<layer number="12" name="Route12" color="20" fill="1" visible="no" active="no"/>
-<layer number="13" name="Route13" color="21" fill="1" visible="no" active="no"/>
-<layer number="14" name="Route14" color="22" fill="1" visible="no" active="no"/>
-<layer number="15" name="Route15" color="23" fill="1" visible="no" active="no"/>
-<layer number="16" name="Bottom" color="1" fill="1" visible="no" active="no"/>
-<layer number="17" name="Pads" color="2" fill="1" visible="no" active="no"/>
-<layer number="18" name="Vias" color="2" fill="1" visible="no" active="no"/>
-<layer number="19" name="Unrouted" color="6" fill="1" visible="no" active="no"/>
-<layer number="20" name="Dimension" color="24" fill="1" visible="no" active="no"/>
-<layer number="21" name="tPlace" color="7" fill="1" visible="no" active="no"/>
-<layer number="22" name="bPlace" color="7" fill="1" visible="no" active="no"/>
-<layer number="23" name="tOrigins" color="15" fill="1" visible="no" active="no"/>
-<layer number="24" name="bOrigins" color="15" fill="1" visible="no" active="no"/>
-<layer number="25" name="tNames" color="7" fill="1" visible="no" active="no"/>
-<layer number="26" name="bNames" color="7" fill="1" visible="no" active="no"/>
-<layer number="27" name="tValues" color="7" fill="1" visible="no" active="no"/>
-<layer number="28" name="bValues" color="7" fill="1" visible="no" active="no"/>
+<layer number="1" name="Top" color="4" fill="1" visible="yes" active="no"/>
+<layer number="2" name="Route2" color="16" fill="1" visible="yes" active="no"/>
+<layer number="3" name="Route3" color="17" fill="1" visible="yes" active="no"/>
+<layer number="4" name="Route4" color="18" fill="1" visible="yes" active="no"/>
+<layer number="5" name="Route5" color="19" fill="1" visible="yes" active="no"/>
+<layer number="6" name="Route6" color="25" fill="1" visible="yes" active="no"/>
+<layer number="7" name="Route7" color="26" fill="1" visible="yes" active="no"/>
+<layer number="8" name="Route8" color="27" fill="1" visible="yes" active="no"/>
+<layer number="9" name="Route9" color="28" fill="1" visible="yes" active="no"/>
+<layer number="10" name="Route10" color="29" fill="1" visible="yes" active="no"/>
+<layer number="11" name="Route11" color="30" fill="1" visible="yes" active="no"/>
+<layer number="12" name="Route12" color="20" fill="1" visible="yes" active="no"/>
+<layer number="13" name="Route13" color="21" fill="1" visible="yes" active="no"/>
+<layer number="14" name="Route14" color="22" fill="1" visible="yes" active="no"/>
+<layer number="15" name="Route15" color="23" fill="1" visible="yes" active="no"/>
+<layer number="16" name="Bottom" color="1" fill="1" visible="yes" active="no"/>
+<layer number="17" name="Pads" color="2" fill="1" visible="yes" active="no"/>
+<layer number="18" name="Vias" color="2" fill="1" visible="yes" active="no"/>
+<layer number="19" name="Unrouted" color="6" fill="1" visible="yes" active="no"/>
+<layer number="20" name="Dimension" color="24" fill="1" visible="yes" active="no"/>
+<layer number="21" name="tPlace" color="7" fill="1" visible="yes" active="no"/>
+<layer number="22" name="bPlace" color="7" fill="1" visible="yes" active="no"/>
+<layer number="23" name="tOrigins" color="15" fill="1" visible="yes" active="no"/>
+<layer number="24" name="bOrigins" color="15" fill="1" visible="yes" active="no"/>
+<layer number="25" name="tNames" color="7" fill="1" visible="yes" active="no"/>
+<layer number="26" name="bNames" color="7" fill="1" visible="yes" active="no"/>
+<layer number="27" name="tValues" color="7" fill="1" visible="yes" active="no"/>
+<layer number="28" name="bValues" color="7" fill="1" visible="yes" active="no"/>
 <layer number="29" name="tStop" color="7" fill="3" visible="no" active="no"/>
 <layer number="30" name="bStop" color="7" fill="6" visible="no" active="no"/>
@@
 <layer number="35" name="tGlue" color="7" fill="4" visible="no" active="no"/>
 <layer number="36" name="bGlue" color="7" fill="5" visible="no" active="no"/>
-<layer number="37" name="tTest" color="7" fill="1" visible="no" active="no"/>
-<layer number="38" name="bTest" color="7" fill="1" visible="no" active="no"/>
+<layer number="37" name="tTest" color="7" fill="1" visible="yes" active="no"/>
+<layer number="38" name="bTest" color="7" fill="1" visible="yes" active="no"/>
 <layer number="39" name="tKeepout" color="4" fill="11" visible="no" active="no"/>
 <layer number="40" name="bKeepout" color="1" fill="11" visible="no" active="no"/>
@@
 <layer number="44" name="Drills" color="7" fill="1" visible="no" active="no"/>
 <layer number="45" name="Holes" color="7" fill="1" visible="no" active="no"/>
-<layer number="46" name="Milling" color="3" fill="1" visible="no" active="no"/>
-<layer number="47" name="Measures" color="7" fill="1" visible="no" active="no"/>
-<layer number="48" name="Document" color="7" fill="1" visible="no" active="no"/>
-<layer number="49" name="Reference" color="7" fill="1" visible="no" active="no"/>
-<layer number="51" name="tDocu" color="7" fill="1" visible="no" active="no"/>
-<layer number="52" name="bDocu" color="7" fill="1" visible="no" active="no"/>
+<layer number="46" name="Milling" color="3" fill="1" visible="yes" active="no"/>
+<layer number="47" name="Measures" color="7" fill="1" visible="yes" active="no"/>
+<layer number="48" name="Document" color="7" fill="1" visible="yes" active="no"/>
+<layer number="49" name="Reference" color="7" fill="1" visible="yes" active="no"/>
+<layer number="51" name="tDocu" color="7" fill="1" visible="yes" active="no"/>
+<layer number="52" name="bDocu" color="7" fill="1" visible="yes" active="no"/>
 <layer number="88" name="SimResults" color="9" fill="1" visible="no" active="yes"/>
 <layer number="89" name="SimProbes" color="9" fill="1" visible="no" active="yes"/>
@@
 <part name="J2" library="BlueHome" deviceset="DCJ200-10-A-XX-X_REVA" device=""/>
 <part name="X4" library="BlueHome" deviceset="2081-1222" device=""/>
-<part name="R53" library="rcl" library_urn="urn:adsk.eagle:library:334" deviceset="R-EU_" device="R1210" package3d_urn="urn:adsk.eagle:package:23554/2"/>
+<part name="R53" library="rcl" library_urn="urn:adsk.eagle:library:334" deviceset="R-EU_" device="R0805" package3d_urn="urn:adsk.eagle:package:23553/2"/>
 <part name="+3V16" library="supply1" library_urn="urn:adsk.eagle:library:371" deviceset="+3V3" device=""/>
 <part name="P+6" library="supply1" library_urn="urn:adsk.eagle:library:371" deviceset="+5V" device=""/>

Commit message: worked on Layout
Parts:
- removed JP10: (no value), jumper:JP1E
- removed JP11: (no value), pinhead:PINHD-1X3
- added C1: (no value), rcl:C-EUC0805
- added SJ1, SJ2: (no value), jumper:SJ
- R62, R65, R68, R69: device rcl:R-EU_R1210 -> rcl:R-EU_R0805
Connections:
- removed net ERROR: R52.1, U3.1B, U3.2B, U3.3B, U3.4B
- removed net JACK: J2.3, R53.1
- net +3V3: now also SJ1.1; no longer JP10.2
- net +5V: now also C1.2
- net AGND: now also C1.1
- net GND: now also JP7.2; no longer JP11.3
- net IO11: now also J2.3, R53.1; no longer JP7.2
- net IO8: now also R52.1, U3.1B, U3.2B, U3.3B, U3.4B
- net N$28: now also SJ1.2; no longer JP10.1
- net RXD: now also SJ2.1; no longer JP11.2
- net TXD: now also SJ2.2; no longer JP11.1
