File: Node#1/Node#1.brd (EAGLE design)
At the start: 260 x 170 mm, 197 parts, among them J1 1757242, J2 DCJ200-10-A-XX-X_REVA, K1 FTR-K1CK005W, K2 FTR-K1CK005W, K3 FTR-K1CK005W, K4 FTR-K1CK005W, U10 ULN2003AIDG4, U11 BLUENRG-232, U12 ACS723LLCTR-40AB-T, U13 RV8564C3, U14 ACS723LLCTR-40AB-T, U2 SEMTECH_SX1503I091TRTSEMTECH_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, U3 MIC4468YWM, U4 LM339ADR, U5 74HC08D,652, U6 SN74LVC1G74DCUR, U7 TMP75BID, U8 IRM-05-5, U9 LMS8117AMP-3.3, X1 2081-1228, X2 2081-1228, X3 2081-1228, X4 2081-1222, Y3 ECS-160-12-36-AGN-TR, Y4 NX2012SA-32.768K-STD-MUB-1

Commit message: Redone Node#1 Layout
Parts:
- removed LED1, LED14, LED15, LED16, LED2, LED3, LED4, LED5, LED6, LED7, LED8, LED9: (no value), led:LED3MM
- removed R10, R19, R20, R21, R22, R23, R24, R25, R26, R27, R28, R29, R30, R31, R32, R33, R34, R35, R36, R37, R38, R7, R8, R9: (no value), rcl:R0805
- removed U$10, U$12, U$13, U$14, U$15, U$16, U$17: BZB984, BlueHome:SOT95P230X110-3N
- added LED18, LED19, LED20, LED21: (no value), led:LED3MM
- added R1, R2, R3, R4, R51, R63, R66, R67: (no value), rcl:R0805
- added U$3, U$4, U$5: BZB984, BlueHome:SOT95P230X110-3N
- moved C26 157.1 mm to (-18.7, 52.5), turned to 180 degrees
- moved C29 145.4 mm to (39.4, 26.0), flipped to the bottom
- moved R11 136.5 mm to (-58.5, 17.3), flipped to the bottom, turned to 90 degrees
- moved LED10 136.1 mm to (-62.4, 17.5), turned to 90 degrees
- moved R14 130.1 mm to (-58.5, 16.0)
- moved R12 129.9 mm to (-60.3, 17.3), flipped to the bottom, turned to 90 degrees
- moved R13 129.0 mm to (-56.8, 17.3), flipped to the bottom, turned to 90 degrees
- moved LED12 128.7 mm to (-75.2, 24.5), turned to 90 degrees
- moved LED13 126.4 mm to (-67.6, 24.5), turned to 90 degrees
- moved LED11 126.0 mm to (-54.7, 17.5), turned to 90 degrees
- moved R18 123.5 mm to (-71.4, 23.0)
- moved R15 122.1 mm to (-71.4, 24.3), flipped to the bottom, turned to 90 degrees
- moved R17 121.9 mm to (-69.6, 24.3), flipped to the bottom, turned to 90 degrees
- moved R16 121.9 mm to (-73.2, 24.3), flipped to the bottom, turned to 90 degrees
- moved JP7 110.2 mm to (-79.8, 25.8), turned to 270 degrees
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Connections:
- removed net E_SHORT: U5.13, U6.5
- removed net E_TEMP: R50.1, U5.12, U7.3
- removed net N$19: LED9.A, R10.2
- removed net N$33: LED1.A, R7.1
- removed net N$49: LED14.A, R19.1
- removed net N$52: LED15.A, R22.2
- removed net N$54: LED2.A, R23.1
- removed net N$58: LED3.A, R26.2
- removed net N$60: LED4.A, R27.1
- removed net N$62: LED5.A, R30.2
- removed net N$64: LED6.A, R31.1
- removed net N$66: LED7.A, R34.2
- removed net N$69: LED8.A, R35.1
- removed net N$72: LED16.A, R38.2
- removed net O_IO10: R28.1
- removed net O_IO11: JP7.2, R29.1, R32.1
- removed net O_IO12: JP7.3, R33.1
- removed net O_IO13: JP7.4, R36.1
- removed net O_IO14: JP7.5, R37.1
- removed net O_IO15: JP7.6
- removed net O_IO8: R24.1
- removed net O_IO9: R25.1
- new net N$1: LED18.A, R1.1
- new net N$10: LED20.A, R51.1
- new net N$11: LED21.A, R67.2
- new net N$2: LED19.A, R4.2
- net ERROR: no longer R49.1, U5.11
- net GND: now also LED18.K, LED19.K, LED20.K, LED21.K, U$3.3, U$4.3, U$5.3; no longer LED1.K, LED14.K, LED15.K, LED16.K, LED2.K, LED3.K, LED4.K, LED5.K, LED6.K, LED7.K, LED8.K, LED9.K, U$10.3, U$12.3, U$13.3, U$14.3, U$15.3, U$16.3, U$17.3
- net IO0: now also R1.2, R2.2, U$3.1; no longer R7.2, R8.2, U$13.1
- net IO1: now also R3.2, R4.1, U$3.2; no longer R10.1, R9.2, U$13.2
- net IO10: now also R50.1, U5.12, U7.3; no longer R27.2, R28.2, U$15.1
- net IO11: now also JP7.2; no longer R29.2, R30.1, U$15.2
- net IO12: now also JP7.3; no longer R31.2, R32.2, U$16.1
- net IO13: now also JP7.4; no longer R33.2, R34.1, U$16.2
- net IO14: now also JP7.5; no longer R35.2, R36.2, U$17.1
- net IO15: now also JP7.6; no longer R37.2, R38.1, U$17.2
- net IO2: now also U$4.1; no longer U$12.1
- net IO3: now also U$4.2; no longer U$12.2
- net IO4: now also U$5.1; no longer U$11.1
- net IO5: now also U$5.2; no longer U$11.2
- net IO6: now also R51.2, R63.2, U$11.1; no longer R19.2, R20.2, U$10.1
- net IO7: now also R66.2, R67.1, U$11.2; no longer R21.2, R22.1, U$10.2
- net IO8: now also R49.1, U5.11; no longer R23.2, R24.2, U$14.1
- net IO9: now also U5.13, U6.5; no longer R25.2, R26.1, U$14.2
- net O_IO0: now also R2.1; no longer R8.1
- net O_IO1: now also R3.1; no longer R9.1
- net O_IO6: now also R63.1; no longer R20.1
- net O_IO7: now also R66.1; no longer R21.1
Routing:
- net V+: track 206.5 -> 46.8 mm, vias 2 -> 0
- net RESETN: track 78.5 -> 194.0 mm, vias 3 -> 5
- net IO10: track 0.00 -> 111.5 mm, vias 0 -> 4
- net SDA: track 107.2 -> 206.1 mm, vias 4 -> 6
- net DIO13: track 60.4 -> 159.3 mm
- net SCL: track 110.1 -> 202.0 mm
- net N$81: track 0.00 -> 90.0 mm, vias 0 -> 2
- net N$80: track 0.00 -> 74.0 mm, vias 0 -> 1
- net +5V: track 274.2 -> 210.5 mm
- net IO9: track 0.00 -> 63.4 mm, vias 0 -> 2
- net N$84: track 0.00 -> 60.1 mm, vias 0 -> 2
- net IO8: track 0.00 -> 59.2 mm, vias 0 -> 2
- net N$39: track 0.00 -> 57.1 mm, vias 0 -> 3
- net N$55: track 0.00 -> 55.0 mm, vias 0 -> 5
- net N$88: track 0.00 -> 46.7 mm, vias 0 -> 2
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Other:
- board size 260 x 170 mm -> 242.7 x 170 mm

Commit message: Arrangement of Node#1 - DC Power Jack
Parts:
- R53: device rcl:R1210 -> rcl:R0805
- moved C35 180.9 mm to (-112.8, 62.6)
- moved C36 180.9 mm to (-110.2, 59.4)
- moved C37 180.9 mm to (-115.3, 59.4)
- moved R68 180.9 mm to (-118.5, 58.2)
- moved R69 180.9 mm to (-115.3, 63.2)
- moved R53 172.4 mm to (-95.8, 31.5)
- moved C34 170.7 mm to (-102.4, 39.4), turned to 270 degrees
- moved X4 163.7 mm to (-83.7, 41.5)
- moved J2 161.6 mm to (-83.4, 51.7), turned to 270 degrees
- moved U$20 151.8 mm to (-71.0, 53.5)
- moved D2 131.2 mm to (-64.1, 35.6)
- moved U$18 131.0 mm to (-59.7, 49.9), turned to 90 degrees
- moved U$21 127.3 mm to (-55.4, 40.1), turned to 0 degrees
- moved C38 127.3 mm to (-56.8, 31.0)
- moved JP8 116.1 mm to (-49.4, 57.5)
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Routing:
- net AGND: track 88.4 -> 8.25 mm, vias 2 -> 1
- net V+: track 46.8 -> 0.00 mm
- net N$42: track 39.9 -> 0.00 mm
- net N$116: track 39.1 -> 0.37 mm, vias 1 -> 0
- net N$13: track 27.3 -> 1.40 mm
- net +5V: track 210.5 -> 185.1 mm
- net L2: track 44.4 -> 65.1 mm
- net CURR_SENS_PWM: track 79.1 -> 59.5 mm, vias 1 -> 0
- net ADC2: track 120.5 -> 101.8 mm
- net N$45: track 15.5 -> 0.00 mm
- net IO11: track 15.3 -> 0.00 mm
- net N$86: track 25.5 -> 40.7 mm
- net N$107: track 15.2 -> 0.13 mm
- net GND: track 22.3 -> 11.8 mm, vias 84 -> 85
- net IO7: track 25.9 -> 15.7 mm
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Other:
- board size 242.7 x 170 mm -> 252.1 x 170.3 mm

Commit message: worked on Layout
Parts:
- removed JP10: (no value), jumper:JP1
- removed JP11: (no value), pinhead:1X03
- added C1: (no value), rcl:C0805
- added SJ1, SJ2: (no value), jumper:SJ
- added U$10, U$14: (no value), holes:3,0
- R62, R65, R68, R69: device rcl:R1210 -> rcl:R0805
- moved R68 58.2 mm to (-64.5, 36.4), flipped to the bottom, turned to 0 degrees
- moved C37 56.7 mm to (-64.5, 34.3), flipped to the bottom, turned to 180 degrees
- moved R69 56.5 mm to (-64.5, 38.6), flipped to the bottom, turned to 180 degrees
- moved C35 55.9 mm to (-61.2, 40.9), flipped to the bottom
- moved C36 52.2 mm to (-61.2, 41.4), turned to 90 degrees
- moved C34 50.4 mm to (-52.3, 45.5), turned to 90 degrees
- moved J1 41.2 mm to (57.3, 4.26)
- moved R53 25.7 mm to (-80.0, 51.8), turned to 90 degrees
- moved VR1 24.9 mm to (-2.79, 63.2), flipped to the top, turned to 180 degrees
- moved U$19 21.5 mm to (55.8, 34.9), turned to 270 degrees
- moved R62 20.0 mm to (49.3, 35.9)
- moved R65 19.9 mm to (49.3, 38.6)
- moved U12 19.6 mm to (47.9, 29.1)
- moved C25 16.7 mm to (50.0, 46.1)
- moved C29 15.9 mm to (50.8, 33.9), turned to 0 degrees
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Connections:
- removed net ERROR: R52.1, U3.2, U3.4, U3.6, U3.9
- removed net JACK: J2.3, R53.1
- net +3V3: now also SJ1.1; no longer JP10.2
- net +5V: now also C1.2
- net AGND: now also C1.1
- net GND: now also JP7.2; no longer JP11.3
- net IO11: now also J2.3, R53.1; no longer JP7.2
- net IO8: now also R52.1, U3.2, U3.4, U3.6, U3.9
- net N$28: now also SJ1.2; no longer JP10.1
- net RXD: now also SJ2.1; no longer JP11.2
- net TXD: now also SJ2.2; no longer JP11.1
Routing:
- net +5V: track 185.1 -> 469.3 mm, vias 1 -> 8
- net +3V3: track 223.5 -> 506.0 mm, vias 9 -> 24
- net AGND: track 8.25 -> 284.0 mm, vias 1 -> 4
- net V+: track 0.00 -> 151.4 mm, vias 0 -> 4
- net IO8: track 59.5 -> 106.0 mm, vias 2 -> 6
- net N$95: track 14.5 -> 53.9 mm
- net N$116: track 0.37 -> 39.7 mm, vias 0 -> 1
- net N$45: track 0.00 -> 33.7 mm, vias 0 -> 1
- net ADC2: track 101.8 -> 134.9 mm
- net N$96: track 0.00 -> 32.3 mm, vias 0 -> 2
- net O_IO2: track 36.9 -> 5.47 mm, vias 1 -> 0
- net N$82: track 5.03 -> 34.2 mm, vias 1 -> 2
- net ERROR: track 22.7 -> 0.00 mm, vias 2 -> 0
- net L2: track 65.1 -> 87.5 mm
- net IO11: track 0.00 -> 21.4 mm, vias 0 -> 2
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Other:
- board size 252.1 x 170.3 mm -> 155 x 71 mm
- board text added: "LÖTSTOPP MASKE"
- board text removed: "STECKER GRÖßE??"
- board text removed: "hoch 71 breit 62"
