File: Node#1/Node#1.brd (EAGLE design)
At the start: 155 x 71 mm, 172 parts, among them J1 1757242, J2 DCJ200-10-A-XX-X_REVA, K1 FTR-K1CK005W, K2 FTR-K1CK005W, K3 FTR-K1CK005W, K4 FTR-K1CK005W, U10 ULN2003AIDG4, U11 BLUENRG-232, U12 ACS723LLCTR-40AB-T, U13 RV8564C3, U14 ACS723LLCTR-40AB-T, U2 SEMTECH_SX1503I091TRTSEMTECH_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, U3 MIC4468YWM, U4 LM339ADR, U5 74HC08D,652, U6 SN74LVC1G74DCUR, U7 TMP75BID, U8 IRM-05-5, U9 LMS8117AMP-3.3, X1 2081-1228, X2 2081-1228, X3 2081-1228, X4 2081-1222, Y3 ECS-160-12-36-AGN-TR, Y4 NX2012SA-32.768K-STD-MUB-1

Commit message: (hopefully) Finished Layout
Parts:
- added U$12, U$13, U$15, U$16, U$17: (no value), holes:3,0
- moved D4 3.28 mm to (26.3, 66.3), flipped to the bottom
- moved K1 2.67 mm to (28.2, 40.5)
- moved JP12 2.55 mm to (17.6, 34.7)
- moved R58 2.41 mm to (27.7, 36.1)
- moved C48 0.25 mm to (19.0, 61.2)
- moved C58 0.25 mm to (25.5, 53.0)
- moved C59 0.25 mm to (26.8, 53.0)
Routing:
- net GND: track 18.2 -> 99.8 mm, vias 74 -> 262
- net ADC2: track 134.9 -> 129.5 mm, vias 3 -> 5
- net N$39: track 49.6 -> 45.8 mm
- net CURR_SENS_RELAY: track 33.9 -> 36.6 mm
- net L1: track 77.9 -> 75.3 mm
- net N$18: track 15.5 -> 17.9 mm
- net DIO14: track 31.2 -> 33.3 mm
- net N$20: track 11.0 -> 13.1 mm, vias 0 -> 1
- net N$29: track 15.2 -> 17.1 mm
- net AGND: track 284.0 -> 282.7 mm
- net DIO13: track 167.5 -> 168.7 mm
- net RESETN: track 203.4 -> 204.6 mm, vias 5 -> 6
- net N$106: track 6.25 -> 7.30 mm
- net N$56: track 40.5 -> 41.5 mm
- net N$105: track 11.8 -> 11.0 mm
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- added copper zone on layer 1, net GND
Other:
- outline, holes or cut-outs redrawn
- board text added: "3.3v Prog"
- board text added: "Firmware Reset"
- board text added: "J-Link"
- board text added: "Power Source"
- board text added: "RESET"
- board text added: "U10"
- board text added: "U11"
- board text added: "U12"
- board text added: "U13"
- board text added: "U14"
- board text added: "U2"
- board text added: "U3"
- board text added: "U4"
- board text added: "U5"
- board text added: "U6"
- board text added: "U7"
- board text added: "U8"
- board text added: "U9"
- board text added: "UART"
- board text removed: "LÖTSTOPP MASKE"

Commit message: finished Layout (again), added Testpoints
Parts:
- added TP1, TP2: PTR1TP20R, testpad:TP20R
Connections:
- net SCL: now also TP1.TP
- net SDA: now also TP2.TP
Routing:
- net SDA: track 216.4 -> 228.1 mm, vias 6 -> 8
- net SCL: track 213.4 -> 218.7 mm, vias 6 -> 7
Changed lines of the file:
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@@
 <element name="U$16" library="holes" package="3,0" value="" x="-88" y="5" smashed="yes" rot="MR0"/>
 <element name="U$17" library="holes" package="3,0" value="" x="-41" y="5" smashed="yes" rot="MR0"/>
+<element name="TP1" library="testpad" package="TP20R" value="PTR1TP20R" x="38.862" y="58.166" smashed="yes" rot="MR0">
+<attribute name="NAME" x="39.862" y="59.216" size="1.27" layer="26" rot="MR0"/>
+<attribute name="TP_SIGNAL_NAME" value="" x="38.862" y="58.166" size="1.778" layer="28" rot="MR0" display="off"/>
+<attribute name="VALUE" x="38.1" y="58.674" size="0.0254" layer="28" rot="MR0"/>
+</element>
+<element name="TP2" library="testpad" package="TP20R" value="PTR1TP20R" x="40.894" y="59.69" smashed="yes">
+<attribute name="NAME" x="39.894" y="60.74" size="1.27" layer="25"/>
+<attribute name="TP_SIGNAL_NAME" value="" x="40.894" y="59.69" size="1.778" layer="27" display="off"/>
+<attribute name="VALUE" x="40.132" y="58.674" size="0.0254" layer="27"/>
+</element>
 </elements>
 <signals>
@@
 <wire x1="30.6159875" y1="60.198" x2="30.956" y2="60.198" width="0.254" layer="1"/>
 <wire x1="30.956" y1="60.198" x2="32.988" y2="58.166" width="0.254" layer="1"/>
-<wire x1="32.988" y1="58.166" x2="34.004" y2="58.166" width="0.254" layer="1"/>
+<wire x1="32.988" y1="58.166" x2="33.782" y2="58.166" width="0.254" layer="1"/>
+<wire x1="33.782" y1="58.166" x2="34.004" y2="58.166" width="0.254" layer="1"/>
 <wire x1="34.004" y1="58.166" x2="34.258" y2="58.42" width="0.254" layer="1"/>
 <wire x1="34.258" y1="58.42" x2="34.22" y2="58.458" width="0.254" layer="1"/>
@@
 <wire x1="-1.905" y1="57.912" x2="-2.286" y2="58.293" width="0.254" layer="16"/>
 <wire x1="-2.286" y1="58.293" x2="-2.286" y2="67.564" width="0.254" layer="16"/>
+<contactref element="TP1" pad="TP"/>
+<wire x1="33.782" y1="58.166" x2="35.052" y2="58.166" width="0.2032" layer="1"/>
+<wire x1="35.052" y1="58.166" x2="35.306" y2="57.912" width="0.2032" layer="1"/>
+<via x="35.306" y="57.912" extent="1-16" drill="0.2032"/>
+<wire x1="38.608" y1="57.912" x2="38.862" y2="58.166" width="0.2032" layer="16"/>
+<wire x1="35.306" y1="57.912" x2="38.608" y2="57.912" width="0.2032" layer="16"/>
 </signal>
 <signal name="SDA">
@@
 <wire x1="27.908" y1="61.976" x2="19.018" y2="61.976" width="0.254" layer="16"/>
 <wire x1="28.924" y1="60.96" x2="30.956" y2="60.96" width="0.254" layer="1"/>
-<wire x1="30.956" y1="60.96" x2="31.8704" y2="60.0456" width="0.254" layer="1"/>
+<wire x1="30.956" y1="60.96" x2="31.48" y2="60.436" width="0.254" layer="1"/>
+<wire x1="31.48" y1="60.436" x2="31.8704" y2="60.0456" width="0.254" layer="1"/>
 <wire x1="31.8704" y1="60.0456" x2="31.8704" y2="59.98906875" width="0.254" layer="1"/>
 <wire x1="31.8704" y1="59.98906875" x2="32.84746875" y2="59.012" width="0.254" layer="1"/>
@@
 <wire x1="1.524" y1="55.88" x2="-0.508" y2="57.912" width="0.254" layer="16"/>
 <wire x1="-0.508" y1="57.912" x2="-1.1808375" y2="57.912" width="0.254" layer="16"/>
+<contactref element="TP2" pad="TP"/>
+<wire x1="40.894" y1="59.69" x2="39.37" y2="59.69" width="0.2032" layer="1"/>
+<via x="39.37" y="59.69" extent="1-16" drill="0.2032"/>
+<via x="31.601896875" y="61.108103125" extent="1-16" drill="0.2032"/>
+<wire x1="39.37" y1="59.69" x2="34.2067625" y2="59.69" width="0.2032" layer="16"/>
+<wire x1="34.2067625" y1="59.69" x2="33.6733625" y2="59.1566" width="0.2032" layer="16"/>
+<wire x1="33.6733625" y1="59.1566" x2="32.5566375" y2="59.1566" width="0.2032" layer="16"/>
+<wire x1="32.5566375" y1="59.1566" x2="31.6926" y2="60.0206375" width="0.2032" layer="16"/>
+<wire x1="31.6926" y1="60.0206375" x2="31.6926" y2="61.0174" width="0.2032" layer="16"/>
+<wire x1="31.6926" y1="61.0174" x2="31.601896875" y2="61.108103125" width="0.2032" layer="16"/>
+<wire x1="31.601896875" y1="61.108103125" x2="31.48" y2="60.98620625" width="0.2032" layer="1"/>
+<wire x1="31.48" y1="60.98620625" x2="31.48" y2="60.436" width="0.2032" layer="1"/>
 </signal>
 <signal name="DIO2">
@@
 <via x="-19.304" y="55.372" extent="1-16" drill="0.2032"/>
 <via x="-15.24" y="58.42" extent="1-16" drill="0.2032"/>
-<via x="38.608" y="57.912" extent="1-16" drill="0.2032"/>
-<via x="39.624" y="59.436" extent="1-16" drill="0.2032"/>
-<via x="40.386" y="60.452" extent="1-16" drill="0.2032"/>
+<via x="37.592" y="56.642" extent="1-16" drill="0.2032"/>
+<via x="39.37" y="60.96" extent="1-16" drill="0.2032"/>
+<via x="40.386" y="57.912" extent="1-16" drill="0.2032"/>
 <via x="35.052" y="55.626" extent="1-16" drill="0.2032"/>
 <via x="33.02" y="55.372" extent="1-16" drill="0.2032"/>
@@
 <via x="42.386" y="42.926" extent="1-16" drill="0.2032" diameter="0.2032"/>
 <via x="33.782" y="55.118" extent="1-16" drill="0.2032"/>
-<via x="36.576" y="57.912" extent="1-16" drill="0.2032"/>
+<via x="36.322" y="55.626" extent="1-16" drill="0.2032"/>
 <via x="-13.462" y="56.642" extent="1-16" drill="0.2032"/>
 <via x="-12.7" y="56.134" extent="1-16" drill="0.2032"/>

Commit message: Last changes for ordering
Routing:
- net GND: track 99.8 -> 105.2 mm, vias 262 -> 250
Other:
- outline, holes or cut-outs redrawn
