File: Node#2/Node#2.brd (EAGLE design)
At the start: 100 x 80 mm, 23 parts, among them IC1 TSL25911FN, J1 68712414522, U2 RV8564C3, U4 TPS63001DRCT

Commit message: Node #2 Update
Parts:
- added C10: 1u, rcl:C0805
- added C11: 100n, rcl:C0805
- added G1, G2, G3: CRAA, battery:CRAA
- added R9: 100, rcl:R0805
Connections:
- new net +3V3: C4.1, C9.1, U4.1
- new net 0V: C10.2, C11.2, C4.2, C9.2, U4.3, U4.9
- new net N$12: C11.1, R9.1, U4.6, U4.7, U4.8
- net GND: no longer C4.2, C9.2, U4.3, U4.9
- net N$8: now also C10.1, R9.2
- net N$9: now also U4.10; no longer U4.8
- net VCC: no longer C4.1, C9.1, U4.1
Changed lines of the file:
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@@
 <element name="C4" library="rcl" package="C0805" value="10u" x="-39.37" y="-142.24"/>
 <element name="C9" library="rcl" package="C0805" value="10u" x="-39.37" y="-148.59"/>
+<element name="R9" library="rcl" package="R0805" value="100" x="-39.37" y="-154.94"/>
+<element name="C10" library="rcl" package="C0805" value="1u" x="-39.37" y="-161.29"/>
+<element name="C11" library="rcl" package="C0805" value="100n" x="-39.37" y="-167.64"/>
+<element name="G1" library="battery" package="CRAA" value="CRAA" x="-13.97" y="-181.61"/>
+<element name="G2" library="battery" package="CRAA" value="CRAA" x="-13.97" y="-199.39"/>
+<element name="G3" library="battery" package="CRAA" value="CRAA" x="-13.97" y="-217.17"/>
 </elements>
 <signals>
@@
 <contactref element="C7" pad="1"/>
 <contactref element="C8" pad="1"/>
-<contactref element="U4" pad="1"/>
-<contactref element="C4" pad="1"/>
-<contactref element="C9" pad="1"/>
-<wire x1="-40.32" y1="-142.24" x2="-40.32" y2="-148.59" width="0" layer="19" extent="1-1"/>
-<wire x1="-40.32" y1="-101.6" x2="-40.32" y2="-142.24" width="0" layer="19" extent="1-1"/>
 <wire x1="-40.32" y1="-95.25" x2="-40.32" y2="-101.6" width="0" layer="19" extent="1-1"/>
 <wire x1="-40.32" y1="-88.9" x2="-40.32" y2="-95.25" width="0" layer="19" extent="1-1"/>
 <wire x1="-40.32" y1="-82.55" x2="-40.32" y2="-88.9" width="0" layer="19" extent="1-1"/>
-<wire x1="-37.0332" y1="-14.2494" x2="-40.32" y2="-82.55" width="0" layer="19" extent="1-1"/>
 </signal>
 <signal name="N$4">
@@
 <signal name="N$8">
 <contactref element="U4" pad="5"/>
-</signal>
-<signal name="N$9">
-<contactref element="U4" pad="8"/>
+<contactref element="R9" pad="2"/>
+<contactref element="C10" pad="1"/>
+<wire x1="-38.42" y1="-154.94" x2="-40.32" y2="-161.29" width="0" layer="19" extent="1-1"/>
+<wire x1="-37.0332" y1="-16.2306" x2="-38.42" y2="-154.94" width="0" layer="19" extent="1-1"/>
 </signal>
 <signal name="GND">
-<contactref element="U4" pad="9"/>
-<contactref element="U4" pad="3"/>
 <contactref element="C5" pad="2"/>
 <contactref element="IC1" pad="3"/>
@@
 <contactref element="C7" pad="2"/>
 <contactref element="C8" pad="2"/>
-<contactref element="C4" pad="2"/>
-<contactref element="C9" pad="2"/>
-<wire x1="-38.42" y1="-142.24" x2="-38.42" y2="-148.59" width="0" layer="19" extent="1-1"/>
-<wire x1="-38.42" y1="-101.6" x2="-38.42" y2="-142.24" width="0" layer="19" extent="1-1"/>
 <wire x1="-38.42" y1="-95.25" x2="-38.42" y2="-101.6" width="0" layer="19" extent="1-1"/>
 <wire x1="-38.42" y1="-88.9" x2="-38.42" y2="-95.25" width="0" layer="19" extent="1-1"/>
 <wire x1="-38.42" y1="-82.55" x2="-38.42" y2="-88.9" width="0" layer="19" extent="1-1"/>
 <wire x1="-37.58" y1="-23.51" x2="-38.42" y2="-82.55" width="0" layer="19" extent="1-1"/>
-<wire x1="-37.0332" y1="-15.24" x2="-37.58" y2="-23.51" width="0" layer="19" extent="1-1"/>
-<wire x1="-34.0868" y1="-14.732" x2="-37.0332" y2="-15.24" width="0" layer="19" extent="1-1"/>
-<wire x1="-29.38" y1="-4.61" x2="-34.0868" y2="-14.732" width="0" layer="19" extent="1-1"/>
+<wire x1="-29.38" y1="-4.61" x2="-37.58" y2="-23.51" width="0" layer="19" extent="1-1"/>
 </signal>
 <signal name="N$10">
@@
 <wire x1="-37.0332" y1="-14.732" x2="-36.15" y2="-134.62" width="0" layer="19" extent="1-1"/>
 </signal>
+<signal name="0V">
+<contactref element="U4" pad="9"/>
+<contactref element="U4" pad="3"/>
+<contactref element="C4" pad="2"/>
+<contactref element="C9" pad="2"/>
+<contactref element="C11" pad="2"/>
+<contactref element="C10" pad="2"/>
+<wire x1="-38.42" y1="-161.29" x2="-38.42" y2="-167.64" width="0" layer="19" extent="1-1"/>
+<wire x1="-38.42" y1="-148.59" x2="-38.42" y2="-161.29" width="0" layer="19" extent="1-1"/>
+<wire x1="-38.42" y1="-142.24" x2="-38.42" y2="-148.59" width="0" layer="19" extent="1-1"/>
+<wire x1="-37.0332" y1="-15.24" x2="-38.42" y2="-142.24" width="0" layer="19" extent="1-1"/>
+<wire x1="-34.0868" y1="-14.732" x2="-37.0332" y2="-15.24" width="0" layer="19" extent="1-1"/>
+</signal>
+<signal name="N$12">
+<contactref element="R9" pad="1"/>
+<contactref element="U4" pad="7"/>
+<contactref element="U4" pad="6"/>
+<contactref element="U4" pad="8"/>
+<contactref element="C11" pad="1"/>
+<wire x1="-40.32" y1="-154.94" x2="-40.32" y2="-167.64" width="0" layer="19" extent="1-1"/>
+<wire x1="-34.0868" y1="-16.2306" x2="-40.32" y2="-154.94" width="0" layer="19" extent="1-1"/>
+<wire x1="-34.0868" y1="-15.748" x2="-34.0868" y2="-16.2306" width="0" layer="19" extent="1-1"/>
+<wire x1="-34.0868" y1="-15.24" x2="-34.0868" y2="-15.748" width="0" layer="19" extent="1-1"/>
+</signal>
+<signal name="+3V3">
+<contactref element="U4" pad="1"/>
+<contactref element="C4" pad="1"/>
+<contactref element="C9" pad="1"/>
+<wire x1="-40.32" y1="-142.24" x2="-40.32" y2="-148.59" width="0" layer="19" extent="1-1"/>
+<wire x1="-37.0332" y1="-14.2494" x2="-40.32" y2="-142.24" width="0" layer="19" extent="1-1"/>
+</signal>
+<signal name="N$9">
+<contactref element="U4" pad="10"/>
+</signal>
 </signals>

Commit message: Node 2 Power, i2 modiefied
Parts:
- added D1: ZPD, diode:DO35Z10
- added Q1: IRF9530, transistor-power:TO220BV
- added R10: 100k, rcl:R0805
Connections:
- removed net 0V: C10.2, C11.2, C4.2, C9.2, U4.3, U4.9
- removed net INT: R3.1, R8.1
- removed net N$8: C10.1, R9.2, U4.5
- removed net VCC: C5.1, C6.1, C7.1, C8.1
- new net +5V: C10.1, D1.C, Q1.D, R9.2, U4.5
- new net GNDA: R10.1, U4.11, U4.3
- new net INT_LI: R3.1
- new net INT_RTC: R8.1
- new net N$14: D1.A, Q1.G, R10.2
- new net N$15: G1.-, G2.-, G3.-
- net +3V3: now also C5.1, C6.1, C7.1, C8.1, U4.10
- net GND: now also C10.2, C11.2, C4.2, C9.2, U4.9
- net N$9: now also G1.+, G2.+, G3.+; no longer U4.10
Changed lines of the file:
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@@
 <layer number="97" name="Info" color="7" fill="1" visible="no" active="no"/>
 <layer number="98" name="Guide" color="6" fill="1" visible="no" active="no"/>
+<layer number="99" name="SpiceOrder" color="5" fill="1" visible="no" active="no"/>
 </layers>
 <board>
@@
 <element name="G2" library="battery" package="CRAA" value="CRAA" x="-13.97" y="-199.39"/>
 <element name="G3" library="battery" package="CRAA" value="CRAA" x="-13.97" y="-217.17"/>
+<element name="Q1" library="transistor-power" package="TO220BV" value="IRF9530" x="-35.56" y="-224.79"/>
+<element name="D1" library="diode" package="DO35Z10" value="ZPD" x="-34.29" y="-236.22"/>
+<element name="R10" library="rcl" package="R0805" value="100k" x="-39.37" y="-242.57"/>
 </elements>
 <signals>
@@
 <wire x1="-40.32" y1="-46.99" x2="-40.32" y2="-120.65" width="0" layer="19" extent="1-1"/>
 </signal>
-<signal name="INT">
-<contactref element="R8" pad="1"/>
+<signal name="INT_LI">
 <contactref element="R3" pad="1"/>
-<wire x1="-40.32" y1="-52.07" x2="-40.32" y2="-127" width="0" layer="19" extent="1-1"/>
 </signal>
 <signal name="N$1">
@@
 <contactref element="IC1" pad="5"/>
 </signal>
-<signal name="VCC">
-<contactref element="C5" pad="1"/>
-<contactref element="C6" pad="1"/>
-<contactref element="C7" pad="1"/>
-<contactref element="C8" pad="1"/>
-<wire x1="-40.32" y1="-95.25" x2="-40.32" y2="-101.6" width="0" layer="19" extent="1-1"/>
-<wire x1="-40.32" y1="-88.9" x2="-40.32" y2="-95.25" width="0" layer="19" extent="1-1"/>
-<wire x1="-40.32" y1="-82.55" x2="-40.32" y2="-88.9" width="0" layer="19" extent="1-1"/>
-</signal>
 <signal name="N$4">
 <contactref element="R8" pad="2"/>
@@
 <wire x1="-31.58" y1="-5.41" x2="-38.42" y2="-114.3" width="0" layer="19" extent="1-1"/>
 </signal>
-<signal name="N$8">
-<contactref element="U4" pad="5"/>
-<contactref element="R9" pad="2"/>
-<contactref element="C10" pad="1"/>
-<wire x1="-38.42" y1="-154.94" x2="-40.32" y2="-161.29" width="0" layer="19" extent="1-1"/>
-<wire x1="-37.0332" y1="-16.2306" x2="-38.42" y2="-154.94" width="0" layer="19" extent="1-1"/>
-</signal>
 <signal name="GND">
 <contactref element="C5" pad="2"/>
-<contactref element="IC1" pad="3"/>
 <contactref element="C6" pad="2"/>
 <contactref element="U2" pad="P$7"/>
 <contactref element="C7" pad="2"/>
 <contactref element="C8" pad="2"/>
+<contactref element="U4" pad="9"/>
+<contactref element="C4" pad="2"/>
+<contactref element="C9" pad="2"/>
+<contactref element="C11" pad="2"/>
+<contactref element="C10" pad="2"/>
+<contactref element="IC1" pad="3"/>
+<wire x1="-38.42" y1="-161.29" x2="-38.42" y2="-167.64" width="0" layer="19" extent="1-1"/>
+<wire x1="-38.42" y1="-148.59" x2="-38.42" y2="-161.29" width="0" layer="19" extent="1-1"/>
+<wire x1="-38.42" y1="-142.24" x2="-38.42" y2="-148.59" width="0" layer="19" extent="1-1"/>
+<wire x1="-38.42" y1="-101.6" x2="-38.42" y2="-142.24" width="0" layer="19" extent="1-1"/>
 <wire x1="-38.42" y1="-95.25" x2="-38.42" y2="-101.6" width="0" layer="19" extent="1-1"/>
 <wire x1="-38.42" y1="-88.9" x2="-38.42" y2="-95.25" width="0" layer="19" extent="1-1"/>
 <wire x1="-38.42" y1="-82.55" x2="-38.42" y2="-88.9" width="0" layer="19" extent="1-1"/>
 <wire x1="-37.58" y1="-23.51" x2="-38.42" y2="-82.55" width="0" layer="19" extent="1-1"/>
-<wire x1="-29.38" y1="-4.61" x2="-37.58" y2="-23.51" width="0" layer="19" extent="1-1"/>
+<wire x1="-34.0868" y1="-14.732" x2="-37.58" y2="-23.51" width="0" layer="19" extent="1-1"/>
+<wire x1="-29.38" y1="-4.61" x2="-34.0868" y2="-14.732" width="0" layer="19" extent="1-1"/>
 </signal>
 <signal name="N$10">
@@
 <contactref element="U4" pad="2"/>
 <wire x1="-37.0332" y1="-14.732" x2="-36.15" y2="-134.62" width="0" layer="19" extent="1-1"/>
-</signal>
-<signal name="0V">
-<contactref element="U4" pad="9"/>
-<contactref element="U4" pad="3"/>
-<contactref element="C4" pad="2"/>
-<contactref element="C9" pad="2"/>
-<contactref element="C11" pad="2"/>
-<contactref element="C10" pad="2"/>
-<wire x1="-38.42" y1="-161.29" x2="-38.42" y2="-167.64" width="0" layer="19" extent="1-1"/>
-<wire x1="-38.42" y1="-148.59" x2="-38.42" y2="-161.29" width="0" layer="19" extent="1-1"/>
-<wire x1="-38.42" y1="-142.24" x2="-38.42" y2="-148.59" width="0" layer="19" extent="1-1"/>
-<wire x1="-37.0332" y1="-15.24" x2="-38.42" y2="-142.24" width="0" layer="19" extent="1-1"/>
-<wire x1="-34.0868" y1="-14.732" x2="-37.0332" y2="-15.24" width="0" layer="19" extent="1-1"/>
 </signal>
 <signal name="N$12">
@@
 <contactref element="C4" pad="1"/>
 <contactref element="C9" pad="1"/>
+<contactref element="C5" pad="1"/>
+<contactref element="C6" pad="1"/>
+<contactref element="C7" pad="1"/>
+<contactref element="C8" pad="1"/>
+<contactref element="U4" pad="10"/>
 <wire x1="-40.32" y1="-142.24" x2="-40.32" y2="-148.59" width="0" layer="19" extent="1-1"/>
-<wire x1="-37.0332" y1="-14.2494" x2="-40.32" y2="-142.24" width="0" layer="19" extent="1-1"/>
+<wire x1="-40.32" y1="-101.6" x2="-40.32" y2="-142.24" width="0" layer="19" extent="1-1"/>
+<wire x1="-40.32" y1="-95.25" x2="-40.32" y2="-101.6" width="0" layer="19" extent="1-1"/>
+<wire x1="-40.32" y1="-88.9" x2="-40.32" y2="-95.25" width="0" layer="19" extent="1-1"/>
+<wire x1="-40.32" y1="-82.55" x2="-40.32" y2="-88.9" width="0" layer="19" extent="1-1"/>
+<wire x1="-37.0332" y1="-14.2494" x2="-40.32" y2="-82.55" width="0" layer="19" extent="1-1"/>
+<wire x1="-34.0868" y1="-14.2494" x2="-37.0332" y2="-14.2494" width="0" layer="19" extent="1-1"/>
+</signal>
+<signal name="+5V">
+<contactref element="U4" pad="5"/>
+<contactref element="R9" pad="2"/>
+<contactref element="C10" pad="1"/>
+<contactref element="Q1" pad="D"/>
+<contactref element="D1" pad="C"/>
+<wire x1="-38.42" y1="-154.94" x2="-40.32" y2="-161.29" width="0" layer="19" extent="1-1"/>
+<wire x1="-35.56" y1="-227.33" x2="-40.32" y2="-161.29" width="0" layer="19" extent="1-1"/>
+<wire x1="-39.37" y1="-236.22" x2="-35.56" y2="-227.33" width="0" layer="19" extent="1-1"/>
+<wire x1="-37.0332" y1="-16.2306" x2="-38.42" y2="-154.94" width="0" layer="19" extent="1-1"/>
+</signal>
+<signal name="INT_RTC">
+<contactref element="R8" pad="1"/>
+</signal>
+<signal name="GNDA">
+<contactref element="U4" pad="3"/>
+<contactref element="U4" pad="11"/>
+<contactref element="R10" pad="1"/>
+<wire x1="-35.56" y1="-15.24" x2="-37.0332" y2="-15.24" width="0" layer="19" extent="1-1"/>
+<wire x1="-40.32" y1="-242.57" x2="-37.0332" y2="-15.24" width="0" layer="19" extent="1-1"/>
 </signal>
 <signal name="N$9">
-<contactref element="U4" pad="10"/>
+<contactref element="G3" pad="+"/>
+<contactref element="G2" pad="+"/>
+<contactref element="G1" pad="+"/>
+<wire x1="-39.37" y1="-186.69" x2="-39.37" y2="-204.47" width="0" layer="19" extent="1-1"/>
+<wire x1="-39.37" y1="-222.25" x2="-39.37" y2="-204.47" width="0" layer="19" extent="1-1"/>
+</signal>
+<signal name="N$14">
+<contactref element="Q1" pad="G"/>
+<contactref element="D1" pad="A"/>
+<contactref element="R10" pad="2"/>
+<wire x1="-29.21" y1="-236.22" x2="-38.42" y2="-242.57" width="0" layer="19" extent="1-1"/>
+<wire x1="-38.1" y1="-227.33" x2="-29.21" y2="-236.22" width="0" layer="19" extent="1-1"/>
+</signal>
+<signal name="N$15">
+<contactref element="G1" pad="-"/>
+<contactref element="G2" pad="-"/>
+<contactref element="G3" pad="-"/>
+<wire x1="11.43" y1="-199.39" x2="11.43" y2="-217.17" width="0" layer="19" extent="1-1"/>
+<wire x1="11.43" y1="-181.61" x2="11.43" y2="-199.39" width="0" layer="19" extent="1-1"/>
 </signal>
 </signals>

Commit message: node2 modified
Parts:
- added U$1: MF-SMDF050, fuse:MF-SMDF050
Connections:
- new net N$8: D1.C, Q1.D, U$1.1
- net +5V: now also U$1.2; no longer D1.C, Q1.D
Changed lines of the file:
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@@
 <element name="D1" library="diode" package="DO35Z10" value="ZPD" x="-34.29" y="-236.22"/>
 <element name="R10" library="rcl" package="R0805" value="100k" x="-39.37" y="-242.57"/>
+<element name="U$1" library="fuse" package="MF-SMDF050" value="MF-SMDF050" x="-46.99" y="-240.03"/>
 </elements>
 <signals>
@@
 <contactref element="R9" pad="2"/>
 <contactref element="C10" pad="1"/>
-<contactref element="Q1" pad="D"/>
-<contactref element="D1" pad="C"/>
+<contactref element="U$1" pad="2"/>
 <wire x1="-38.42" y1="-154.94" x2="-40.32" y2="-161.29" width="0" layer="19" extent="1-1"/>
-<wire x1="-35.56" y1="-227.33" x2="-40.32" y2="-161.29" width="0" layer="19" extent="1-1"/>
-<wire x1="-39.37" y1="-236.22" x2="-35.56" y2="-227.33" width="0" layer="19" extent="1-1"/>
+<wire x1="-44.54" y1="-240.03" x2="-40.32" y2="-161.29" width="0" layer="19" extent="1-1"/>
 <wire x1="-37.0332" y1="-16.2306" x2="-38.42" y2="-154.94" width="0" layer="19" extent="1-1"/>
 </signal>
@@
 <wire x1="11.43" y1="-181.61" x2="11.43" y2="-199.39" width="0" layer="19" extent="1-1"/>
 </signal>
+<signal name="N$8">
+<contactref element="Q1" pad="D"/>
+<contactref element="D1" pad="C"/>
+<contactref element="U$1" pad="1"/>
+<wire x1="-39.37" y1="-236.22" x2="-49.44" y2="-240.03" width="0" layer="19" extent="1-1"/>
+<wire x1="-35.56" y1="-227.33" x2="-39.37" y2="-236.22" width="0" layer="19" extent="1-1"/>
+</signal>
 </signals>

Commit message: node 2 display
Parts:
- removed LS1: CMS-181325-078S, BlueHome:SPKR_CMS-181325-078S
- added !!!MBR0530!!!, !!!MBR0530!!!1, !!!MBR0530!!!2: PD3S160, diode:POWERDI323
- added !!!SI1308EDL!!!: (no value), zetex:SOT-23
- added C12, C14: 1u, rcl:C0805
- added C13, C15: 100n, rcl:C0805
- added C16, C17: 100nF, rcl:C0805
- added C18: 1nF_5%, rcl:C0805
- added C19: 0.1µF, rcl:C0805
- added C20, C21, C22, C23, C28, C30, C33: 1µF, rcl:C0805
- added C24, C25, C27, C29, C31: 10µF, rcl:C0805
- added C26: 4.7µF, rcl:C0805
- added C32: 2.2µF, rcl:C0805
- added HM1: HDC2080DMBR, BlueHome:SON100P300X300X80-7N
- added L2: 10µH, rcl:L1812
- added MK1: ICS-40180, BlueHome:MIC_ICS-40180
- added R11, R12, R13, R14: 10k, rcl:R0805
- added R15: 470m, rcl:R0805
- added U$2: SX8635, BlueHome:QFN-32
- moved R8 151.9 mm to (-54.6, -278.1)
Connections:
- net INT_LI renamed INT_TSL
- new net ADC: C32.2
- new net BS: J1.8
- new net BUSY_N: J1.9
- new net CSB: J1.12
- new net DC: J1.11
- new net GDR: !!!SI1308EDL!!!.3, J1.2
- new net INT_HDC: HM1.4
- new net N$13: HM1.1, R11.2
- new net N$16: R13.2, U$2.15
- new net N$17: R14.2, U$2.16
- new net N$18: C16.2, U$2.27
- new net N$19: C17.2, U$2.30
- new net N$20: C18.2, U$2.12
- new net N$21: C18.1, U$2.11
- new net N$22: C32.1, MK1.1
- new net N$23: !!!MBR0530!!!.A, !!!SI1308EDL!!!.1, C26.1, L2.2
- new net N$24: !!!MBR0530!!!1.A, !!!MBR0530!!!2.C, C26.2
- new net N$26: C31.2, C33.2, MK1.5
- new net RESE: !!!SI1308EDL!!!.2, J1.3, R15.2
- new net RESET: U$2.29
- new net RST_N: J1.10
- new net SCL*: J1.13
- new net SDA*: J1.14
- new net TSCL: J1.6
- new net TSDA: J1.7
- new net VCOM: C19.2, J1.24
- new net VDD_18V: C20.2, J1.18
- new net VGH: !!!MBR0530!!!.C, C27.2, C30.2, J1.21
- new net VGL: !!!MBR0530!!!2.A, C28.2, C29.2, J1.23
- new net VOTP: C23.1, J1.19
- new net VSH: C21.2, J1.20
- new net VSHR: C22.2, J1.22
- new net VSL: J1.5
- new net VSLR: J1.4
- new net VSS: C19.1, C20.1, C21.1, C22.1, C23.2, J1.17
- net +3V3: now also C12.1, C13.1, C14.1, C15.1, C16.1, C17.1, C24.1, C25.1, C31.1, C33.1, HM1.5, IC1.5, J1.15, J1.16, L2.1, U$2.13
- net GND: now also !!!MBR0530!!!1.C, C12.2, C13.2, C14.2, C15.2, C24.2, C25.2, C27.1, C28.1, C29.1, C30.1, HM1.2, MK1.2, MK1.3, MK1.4, R15.1, U$2.19, U$2.24, U$2.28, U$2.EP
- net INT_RTC: now also R8.2; no longer R8.1
- net N$4: now also R8.1; no longer R8.2
- net N$6: now also HM1.6, R12.2; no longer IC1.5
- net SCL: now also R12.1, R13.1
- net SDA: now also R11.1, R14.1

Commit message: restored
Parts:
- removed !!!MBR0530!!!, !!!MBR0530!!!1, !!!MBR0530!!!2: PD3S160, diode:POWERDI323
- removed !!!SI1308EDL!!!: (no value), zetex:SOT-23
- added D5, D6, D7: MBR0530, BlueHome:SOD3716X135N
- added Q2: SI1308EDL-T1-GE3, BlueHome:SOT65P210X110-3N
- added R16: 10k, rcl:R0805
- C26: value 4.7µF -> 0.1µF
- L2: value 10µH -> 68µH
Connections:
- net GDR: now also Q2.1, R16.2; no longer !!!SI1308EDL!!!.3
- net GND: now also D5.1, R16.1; no longer !!!MBR0530!!!1.C
- net N$23: now also D6.2, Q2.3; no longer !!!MBR0530!!!.A, !!!SI1308EDL!!!.1
- net N$24: now also D5.2, D7.1; no longer !!!MBR0530!!!1.A, !!!MBR0530!!!2.C
- net N$8: now also Q1.S; no longer Q1.D
- net N$9: now also Q1.D
- net RESE: now also Q2.2; no longer !!!SI1308EDL!!!.2
- net VGH: now also D6.1; no longer !!!MBR0530!!!.C
- net VGL: now also D7.2; no longer !!!MBR0530!!!2.A
