File: Node#2/Node#2.brd (EAGLE design)
At the start: 100 x 80 mm, 68 parts, among them IC1 TSL25911FN, J1 68712414522, Q1 IRF9530, Q2 SI1308EDL-T1-GE3, U2 RV8564C3, U4 TPS63001DRCT

Commit message: bi-colour_leds
Parts:
- added LED1, LED2, LED3, LED4, LED5, LED6: 156125YV73000, BlueHome:156125YV73000
Connections:
- new net LED0: LED1.1, LED2.1, LED3.1, LED4.1, LED5.1, LED6.1, U$2.17
- new net LED1: LED1.2, U$2.18
- new net LED2: LED2.2, U$2.20
- new net LED3: LED3.2, U$2.21
- new net LED4: LED4.2, U$2.22
- new net LED5: LED5.2, U$2.23
- new net LED6: LED6.2
- new net N$25: LED1.3, LED1.4, LED2.3, LED2.4
- new net N$27: LED3.3, LED3.4, LED4.3, LED4.4
- new net N$30: LED5.3, LED5.4, LED6.3, LED6.4
- new net N$34: U$2.25
- new net N$35: U$2.26
Changed lines of the file:
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@@
 <attribute name="DESCRIPTION" value="ON SEMICONDUCTOR - MBR0530 - DIODE, SCHOTTKY, 0.5A, 30V, SOD-123" x="-57.15" y="-506.73" size="1.778" layer="27" display="off"/>
+</element>
+<element name="LED1" library="BlueHome" package="156125YV73000" value="156125YV73000" x="-57.15" y="-510.54">
+<attribute name="HEIGHT" value="0.8mm" x="-57.15" y="-510.54" size="1.778" layer="27" display="off"/>
+<attribute name="MANUFACTURER_NAME" value="Wurth Elektronik" x="-57.15" y="-510.54" size="1.778" layer="27" display="off"/>
+<attribute name="MOUSER_PART_NUMBER" value="710-156125YV73000" x="-57.15" y="-510.54" size="1.778" layer="27" display="off"/>
+<attribute name="MANUFACTURER_PART_NUMBER" value="156125YV73000" x="-57.15" y="-510.54" size="1.778" layer="27" display="off"/>
+<attribute name="DESCRIPTION" value="Standard LEDs - SMD WL-SBRW SMD 1205 YBG 592/573nm" x="-57.15" y="-510.54" size="1.778" layer="27" display="off"/>
+</element>
+<element name="LED2" library="BlueHome" package="156125YV73000" value="156125YV73000" x="-59.69" y="-515.62">
+<attribute name="HEIGHT" value="0.8mm" x="-59.69" y="-515.62" size="1.778" layer="27" display="off"/>
+<attribute name="MANUFACTURER_NAME" value="Wurth Elektronik" x="-59.69" y="-515.62" size="1.778" layer="27" display="off"/>
+<attribute name="MOUSER_PART_NUMBER" value="710-156125YV73000" x="-59.69" y="-515.62" size="1.778" layer="27" display="off"/>
+<attribute name="MANUFACTURER_PART_NUMBER" value="156125YV73000" x="-59.69" y="-515.62" size="1.778" layer="27" display="off"/>
+<attribute name="DESCRIPTION" value="Standard LEDs - SMD WL-SBRW SMD 1205 YBG 592/573nm" x="-59.69" y="-515.62" size="1.778" layer="27" display="off"/>
+</element>
+<element name="LED3" library="BlueHome" package="156125YV73000" value="156125YV73000" x="-59.69" y="-520.7">
+<attribute name="HEIGHT" value="0.8mm" x="-62.23" y="-520.7" size="1.778" layer="27" display="off"/>
+<attribute name="MANUFACTURER_NAME" value="Wurth Elektronik" x="-62.23" y="-520.7" size="1.778" layer="27" display="off"/>
+<attribute name="MOUSER_PART_NUMBER" value="710-156125YV73000" x="-62.23" y="-520.7" size="1.778" layer="27" display="off"/>
+<attribute name="MANUFACTURER_PART_NUMBER" value="156125YV73000" x="-62.23" y="-520.7" size="1.778" layer="27" display="off"/>
+<attribute name="DESCRIPTION" value="Standard LEDs - SMD WL-SBRW SMD 1205 YBG 592/573nm" x="-62.23" y="-520.7" size="1.778" layer="27" display="off"/>
+</element>
+<element name="LED4" library="BlueHome" package="156125YV73000" value="156125YV73000" x="-59.69" y="-525.78">
+<attribute name="HEIGHT" value="0.8mm" x="-64.77" y="-525.78" size="1.778" layer="27" display="off"/>
+<attribute name="MANUFACTURER_NAME" value="Wurth Elektronik" x="-64.77" y="-525.78" size="1.778" layer="27" display="off"/>
+<attribute name="MOUSER_PART_NUMBER" value="710-156125YV73000" x="-64.77" y="-525.78" size="1.778" layer="27" display="off"/>
+<attribute name="MANUFACTURER_PART_NUMBER" value="156125YV73000" x="-64.77" y="-525.78" size="1.778" layer="27" display="off"/>
+<attribute name="DESCRIPTION" value="Standard LEDs - SMD WL-SBRW SMD 1205 YBG 592/573nm" x="-64.77" y="-525.78" size="1.778" layer="27" display="off"/>
+</element>
+<element name="LED5" library="BlueHome" package="156125YV73000" value="156125YV73000" x="-59.69" y="-530.86">
+<attribute name="HEIGHT" value="0.8mm" x="-62.23" y="-530.86" size="1.778" layer="27" display="off"/>
+<attribute name="MANUFACTURER_NAME" value="Wurth Elektronik" x="-62.23" y="-530.86" size="1.778" layer="27" display="off"/>
+<attribute name="MOUSER_PART_NUMBER" value="710-156125YV73000" x="-62.23" y="-530.86" size="1.778" layer="27" display="off"/>
+<attribute name="MANUFACTURER_PART_NUMBER" value="156125YV73000" x="-62.23" y="-530.86" size="1.778" layer="27" display="off"/>
+<attribute name="DESCRIPTION" value="Standard LEDs - SMD WL-SBRW SMD 1205 YBG 592/573nm" x="-62.23" y="-530.86" size="1.778" layer="27" display="off"/>
+</element>
+<element name="LED6" library="BlueHome" package="156125YV73000" value="156125YV73000" x="-59.69" y="-535.94">
+<attribute name="HEIGHT" value="0.8mm" x="-64.77" y="-535.94" size="1.778" layer="27" display="off"/>
+<attribute name="MANUFACTURER_NAME" value="Wurth Elektronik" x="-64.77" y="-535.94" size="1.778" layer="27" display="off"/>
+<attribute name="MOUSER_PART_NUMBER" value="710-156125YV73000" x="-64.77" y="-535.94" size="1.778" layer="27" display="off"/>
+<attribute name="MANUFACTURER_PART_NUMBER" value="156125YV73000" x="-64.77" y="-535.94" size="1.778" layer="27" display="off"/>
+<attribute name="DESCRIPTION" value="Standard LEDs - SMD WL-SBRW SMD 1205 YBG 592/573nm" x="-64.77" y="-535.94" size="1.778" layer="27" display="off"/>
 </element>
 </elements>
@@
 <contactref element="C32" pad="2"/>
 </signal>
+<signal name="N$25">
+<contactref element="LED2" pad="3"/>
+<contactref element="LED2" pad="4"/>
+<contactref element="LED1" pad="4"/>
+<contactref element="LED1" pad="3"/>
+<wire x1="-58.14" y1="-515.045" x2="-58.14" y2="-516.195" width="0" layer="19" extent="1-1"/>
+<wire x1="-55.6" y1="-511.115" x2="-58.14" y2="-515.045" width="0" layer="19" extent="1-1"/>
+<wire x1="-55.6" y1="-509.965" x2="-55.6" y2="-511.115" width="0" layer="19" extent="1-1"/>
+</signal>
+<signal name="LED0">
+<contactref element="U$2" pad="17"/>
+<contactref element="LED1" pad="1"/>
+<contactref element="LED2" pad="1"/>
+<contactref element="LED3" pad="1"/>
+<contactref element="LED4" pad="1"/>
+<contactref element="LED5" pad="1"/>
+<contactref element="LED6" pad="1"/>
+<wire x1="-61.24" y1="-531.435" x2="-61.24" y2="-536.515" width="0" layer="19" extent="1-1"/>
+<wire x1="-61.24" y1="-526.355" x2="-61.24" y2="-531.435" width="0" layer="19" extent="1-1"/>
+<wire x1="-61.24" y1="-521.275" x2="-61.24" y2="-526.355" width="0" layer="19" extent="1-1"/>
+<wire x1="-61.24" y1="-516.195" x2="-61.24" y2="-521.275" width="0" layer="19" extent="1-1"/>
+<wire x1="-58.7" y1="-511.115" x2="-61.24" y2="-516.195" width="0" layer="19" extent="1-1"/>
+<wire x1="-51.59" y1="-281.98" x2="-58.7" y2="-511.115" width="0" layer="19" extent="1-1"/>
+</signal>
+<signal name="LED1">
+<contactref element="U$2" pad="18"/>
+<contactref element="LED1" pad="2"/>
+<wire x1="-58.7" y1="-509.965" x2="-52.09" y2="-281.98" width="0" layer="19" extent="1-1"/>
+</signal>
+<signal name="LED2">
+<contactref element="U$2" pad="20"/>
+<contactref element="LED2" pad="2"/>
+<wire x1="-61.24" y1="-515.045" x2="-53.09" y2="-281.98" width="0" layer="19" extent="1-1"/>
+</signal>
+<signal name="LED3">
+<contactref element="U$2" pad="21"/>
+<contactref element="LED3" pad="2"/>
+<wire x1="-61.24" y1="-520.125" x2="-53.59" y2="-281.98" width="0" layer="19" extent="1-1"/>
+</signal>
+<signal name="LED4">
+<contactref element="U$2" pad="22"/>
+<contactref element="LED4" pad="2"/>
+<wire x1="-61.24" y1="-525.205" x2="-54.09" y2="-281.98" width="0" layer="19" extent="1-1"/>
+</signal>
+<signal name="LED5">
+<contactref element="U$2" pad="23"/>
+<contactref element="LED5" pad="2"/>
+<wire x1="-61.24" y1="-530.285" x2="-54.59" y2="-281.98" width="0" layer="19" extent="1-1"/>
+</signal>
+<signal name="N$34">
+<contactref element="U$2" pad="25"/>
+</signal>
+<signal name="N$35">
+<contactref element="U$2" pad="26"/>
+</signal>
+<signal name="N$27">
+<contactref element="LED4" pad="3"/>
+<contactref element="LED4" pad="4"/>
+<contactref element="LED3" pad="4"/>
+<contactref element="LED3" pad="3"/>
+<wire x1="-58.14" y1="-525.205" x2="-58.14" y2="-526.355" width="0" layer="19" extent="1-1"/>
+<wire x1="-58.14" y1="-521.275" x2="-58.14" y2="-525.205" width="0" layer="19" extent="1-1"/>
+<wire x1="-58.14" y1="-520.125" x2="-58.14" y2="-521.275" width="0" layer="19" extent="1-1"/>
+</signal>
+<signal name="N$30">
+<contactref element="LED6" pad="3"/>
+<contactref element="LED6" pad="4"/>
+<contactref element="LED5" pad="4"/>
+<contactref element="LED5" pad="3"/>
+<wire x1="-58.14" y1="-535.365" x2="-58.14" y2="-536.515" width="0" layer="19" extent="1-1"/>
+<wire x1="-58.14" y1="-531.435" x2="-58.14" y2="-535.365" width="0" layer="19" extent="1-1"/>
+<wire x1="-58.14" y1="-530.285" x2="-58.14" y2="-531.435" width="0" layer="19" extent="1-1"/>
+</signal>
+<signal name="LED6">
+<contactref element="LED6" pad="2"/>
+</signal>
 </signals>

Commit message: small changes
Parts:
- removed C1: (no value), rcl:C0805
- removed C2: 1u, rcl:C0805
- removed C3: 100n, rcl:C0805
- removed R11, R12, R13, R14, R2, R4, R6, R7: 10k, rcl:R0805
- added R17: 1.5M, rcl:R0805
- added R18: 10k, rcl:R0805
- added U$3, U$4, U$5, U$6, U$7: TOUCH_BUTTON, BlueHome:TOUCH_BUTTON
- added U$8: WHEEL, BlueHome:WHEEL
- R1: value (none) -> 10k
- R3, R8: value 10k -> 4.7k
- R5: value 10k -> 1M
- moved R1 653.3 mm to (-64.8, -689.6)
- moved R3 644.4 mm to (-64.8, -696.0)
- moved R5 569.5 mm to (-64.8, -676.9)
- moved R8 424.3 mm to (-64.8, -702.3)
Connections:
- net ADC renamed ADC1
- net GNDA renamed V-
- removed net N$1: IC1.6, R4.2
- removed net N$13: HM1.1, R11.2
- removed net N$16: R13.2, U$2.15
- removed net N$17: R14.2, U$2.16
- removed net N$2: IC1.1, R2.2
- removed net N$25: LED1.3, LED1.4, LED2.3, LED2.4
- removed net N$27: LED3.3, LED3.4, LED4.3, LED4.4
- removed net N$3: IC1.2, R3.2
- removed net N$30: LED5.3, LED5.4, LED6.3, LED6.4
- removed net N$4: R8.1, U2.P$6
- removed net N$5: R7.2, U2.P$4
- removed net N$6: HM1.6, R12.2
- removed net N$7: R6.2, U2.P$5
- new net ADC2: R17.2, R5.1
- new net INT_SX: U$2.14
- new net N$28: U$2.32, U$3.P$1
- new net N$29: U$2.1, U$4.P$1
- new net N$31: U$2.2, U$5.P$1
- new net N$32: U$2.3, U$6.P$1
- new net N$33: U$2.31, U$7.P$1
- new net SEG1: U$2.4, U$8.SEG1
- new net SEG2: U$2.5, U$8.SEG2
- new net SEG3: U$2.6, U$8.SEG3
- new net SEG4: U$2.7, U$8.SEG4
- new net V+: C10.1, R9.2, U4.5
- net +3V3: now also LED1.3, LED1.4, LED2.3, LED2.4, LED3.3, LED3.4, LED4.3, LED4.4, LED5.3, LED5.4, LED6.3, LED6.4, R1.2, R3.2, R8.2
- net +5V: now also R5.2; no longer C10.1, R9.2, U4.5
- net CSB: now also R1.1, R18.2
- net GND: now also HM1.3, R17.1, R18.1, U2.P$1
- net INT_RTC: now also U2.P$6; no longer R8.2
- net INT_TSL: now also IC1.2; no longer R3.1
- net SCL: now also HM1.6, IC1.1, U$2.15, U2.P$4; no longer R12.1, R13.1, R2.1, R7.1
- net SDA: now also HM1.1, IC1.6, U$2.16, U2.P$5; no longer R11.1, R14.1, R4.1, R6.1
- net TSCL: now also R8.1
- net TSDA: now also R3.1
Routing:
- added copper zone on layer 1, net N$1

Commit message: node2 spi, rtc
Parts:
- removed Q1: IRF9530, transistor-power:TO220BV
- added !!!FDN304PZ!!!: BSS84, transistor-small-signal:SOT23
- added C1, C2: 1µF, rcl:C0805
- added C3: 100mF, rcl:C050-055X075
- added D2: MUR150RL, diode:DO41-10
- C26: value 0.1µF -> 4.7µF
- L1: device rcl:L1812 -> rcl:L4532P
- L2: value 68µH -> 10µH
Connections:
- net CSB renamed CS
- removed net SCL*: J1.13
- removed net SDA*: J1.14
- new net +3V3_RTC: C3.1, C7.2, C8.2, D2.C, U2.P$2
- new net MOSI: J1.14, R3.1
- new net SCLK: J1.13, R8.1
- net +3V3: now also D2.A; no longer C7.1, C8.1
- net GND: now also C1.1, C2.2, C3.2, C7.1, C8.1; no longer C7.2, C8.2
- net N$14: now also !!!FDN304PZ!!!.1; no longer Q1.G
- net N$8: now also !!!FDN304PZ!!!.2; no longer Q1.S
- net N$9: now also !!!FDN304PZ!!!.3; no longer Q1.D
- net SDA: no longer U2.P$2
- net TSCL: no longer R8.1
- net TSDA: no longer R3.1
- net VSL: now also C1.2
- net VSLR: now also C2.1
