File: Node#2/Node#2.sch (EAGLE design)
At the start: 23 parts, among them IC1 TSL25911FN, J1 68712414522, U2 RV8564C3, U4 TPS63001DRCT

Commit message: Node #2 Update
Parts:
- added C10: 1u, rcl:C-EUC0805
- added C11: 100n, rcl:C-EUC0805
- added G1, G2, G3: CRAA, battery:CRAA
- added R9: 100, rcl:R-EU_R0805
Connections:
- new net +3V3: C4.1, C9.1, U4.VOUT
- new net 0V: C10.2, C11.2, C4.2, C9.2, U4.GND, U4.PGND
- new net N$12: C11.1, R9.1, U4.EN, U4.PS/SYNC, U4.VINA
- net GND: no longer C4.2, C9.2, U4.GND, U4.PGND
- net N$8: now also C10.1, R9.2
- net N$9: now also U4.FB; no longer U4.VINA
- net VCC: no longer C4.1, C9.1, U4.VOUT
Changed lines of the file:
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@@
 <part name="C4" library="rcl" deviceset="C-EU" device="C0805" value="10u"/>
 <part name="C9" library="rcl" deviceset="C-EU" device="C0805" value="10u"/>
+<part name="+3V1" library="supply1" deviceset="+3V3" device=""/>
+<part name="GND1" library="supply1" deviceset="0V" device=""/>
+<part name="R9" library="rcl" deviceset="R-EU_" device="R0805" value="100"/>
+<part name="C10" library="rcl" deviceset="C-EU" device="C0805" value="1u"/>
+<part name="C11" library="rcl" deviceset="C-EU" device="C0805" value="100n"/>
+<part name="G1" library="battery" deviceset="CRAA" device=""/>
+<part name="G2" library="battery" deviceset="CRAA" device=""/>
+<part name="G3" library="battery" deviceset="CRAA" device=""/>
 </parts>
 <sheets>
@@
 <instance part="C4" gate="G$1" x="149.86" y="170.18"/>
 <instance part="C9" gate="G$1" x="162.56" y="170.18"/>
+<instance part="+3V1" gate="G$1" x="170.18" y="185.42"/>
+<instance part="GND1" gate="1" x="162.56" y="134.62"/>
+<instance part="R9" gate="G$1" x="83.82" y="172.72" rot="R90"/>
+<instance part="C10" gate="G$1" x="71.12" y="167.64"/>
+<instance part="C11" gate="G$1" x="83.82" y="162.56"/>
+<instance part="G1" gate="G$1" x="17.78" y="165.1" rot="R90"/>
+<instance part="G2" gate="G$1" x="5.08" y="165.1" rot="R90"/>
+<instance part="G3" gate="G$1" x="-7.62" y="165.1" rot="R90"/>
 </instances>
 <busses>
@@
 <junction x="187.96" y="68.58"/>
 </segment>
-<segment>
-<pinref part="U4" gate="A" pin="VOUT"/>
-<wire x1="142.24" y1="180.34" x2="149.86" y2="180.34" width="0.1524" layer="91"/>
-<label x="167.64" y="180.34" size="1.778" layer="95"/>
-<pinref part="C4" gate="G$1" pin="1"/>
-<wire x1="149.86" y1="180.34" x2="162.56" y2="180.34" width="0.1524" layer="91"/>
-<wire x1="162.56" y1="180.34" x2="167.64" y2="180.34" width="0.1524" layer="91"/>
-<wire x1="149.86" y1="172.72" x2="149.86" y2="180.34" width="0.1524" layer="91"/>
-<junction x="149.86" y="180.34"/>
-<pinref part="C9" gate="G$1" pin="1"/>
-<wire x1="162.56" y1="172.72" x2="162.56" y2="180.34" width="0.1524" layer="91"/>
-<junction x="162.56" y="180.34"/>
-</segment>
 </net>
 <net name="N$4" class="0">
@@
 <segment>
 <pinref part="U4" gate="A" pin="VIN"/>
-<wire x1="106.68" y1="180.34" x2="78.74" y2="180.34" width="0.1524" layer="91"/>
-</segment>
-</net>
-<net name="N$9" class="0">
-<segment>
-<pinref part="U4" gate="A" pin="VINA"/>
-<wire x1="106.68" y1="177.8" x2="78.74" y2="177.8" width="0.1524" layer="91"/>
+<wire x1="106.68" y1="180.34" x2="83.82" y2="180.34" width="0.1524" layer="91"/>
+<pinref part="R9" gate="G$1" pin="2"/>
+<wire x1="83.82" y1="177.8" x2="83.82" y2="180.34" width="0.1524" layer="91"/>
+<junction x="83.82" y="180.34"/>
+<wire x1="83.82" y1="180.34" x2="71.12" y2="180.34" width="0.1524" layer="91"/>
+<pinref part="C10" gate="G$1" pin="1"/>
+<wire x1="71.12" y1="180.34" x2="71.12" y2="170.18" width="0.1524" layer="91"/>
+<wire x1="71.12" y1="180.34" x2="55.88" y2="180.34" width="0.1524" layer="91"/>
+<junction x="71.12" y="180.34"/>
 </segment>
 </net>
 <net name="GND" class="0">
-<segment>
-<pinref part="U4" gate="A" pin="GND"/>
-<wire x1="106.68" y1="154.94" x2="101.6" y2="154.94" width="0.1524" layer="91"/>
-<wire x1="101.6" y1="154.94" x2="101.6" y2="152.4" width="0.1524" layer="91"/>
-<wire x1="101.6" y1="152.4" x2="101.6" y2="139.7" width="0.1524" layer="91"/>
-<wire x1="101.6" y1="139.7" x2="149.86" y2="139.7" width="0.1524" layer="91"/>
-<pinref part="U4" gate="A" pin="PGND"/>
-<wire x1="149.86" y1="139.7" x2="162.56" y2="139.7" width="0.1524" layer="91"/>
-<wire x1="162.56" y1="139.7" x2="167.64" y2="139.7" width="0.1524" layer="91"/>
-<wire x1="106.68" y1="152.4" x2="101.6" y2="152.4" width="0.1524" layer="91"/>
-<junction x="101.6" y="152.4"/>
-<label x="167.64" y="139.7" size="1.778" layer="95"/>
-<pinref part="C4" gate="G$1" pin="2"/>
-<wire x1="149.86" y1="165.1" x2="149.86" y2="139.7" width="0.1524" layer="91"/>
-<junction x="149.86" y="139.7"/>
-<pinref part="C9" gate="G$1" pin="2"/>
-<wire x1="162.56" y1="165.1" x2="162.56" y2="139.7" width="0.1524" layer="91"/>
-<junction x="162.56" y="139.7"/>
-</segment>
 <segment>
 <wire x1="200.66" y1="-7.62" x2="200.66" y2="12.7" width="0.1524" layer="91"/>
@@
 </segment>
 </net>
+<net name="0V" class="0">
+<segment>
+<pinref part="U4" gate="A" pin="GND"/>
+<wire x1="106.68" y1="154.94" x2="101.6" y2="154.94" width="0.1524" layer="91"/>
+<wire x1="101.6" y1="154.94" x2="101.6" y2="152.4" width="0.1524" layer="91"/>
+<wire x1="101.6" y1="152.4" x2="101.6" y2="139.7" width="0.1524" layer="91"/>
+<wire x1="101.6" y1="139.7" x2="149.86" y2="139.7" width="0.1524" layer="91"/>
+<pinref part="U4" gate="A" pin="PGND"/>
+<wire x1="149.86" y1="139.7" x2="162.56" y2="139.7" width="0.1524" layer="91"/>
+<wire x1="162.56" y1="139.7" x2="162.56" y2="137.16" width="0.1524" layer="91"/>
+<wire x1="106.68" y1="152.4" x2="101.6" y2="152.4" width="0.1524" layer="91"/>
+<junction x="101.6" y="152.4"/>
+<label x="165.1" y="137.16" size="1.778" layer="95"/>
+<pinref part="C4" gate="G$1" pin="2"/>
+<wire x1="149.86" y1="165.1" x2="149.86" y2="139.7" width="0.1524" layer="91"/>
+<junction x="149.86" y="139.7"/>
+<pinref part="C9" gate="G$1" pin="2"/>
+<wire x1="162.56" y1="165.1" x2="162.56" y2="139.7" width="0.1524" layer="91"/>
+<junction x="162.56" y="139.7"/>
+<pinref part="GND1" gate="1" pin="0V"/>
+<pinref part="C11" gate="G$1" pin="2"/>
+<wire x1="83.82" y1="157.48" x2="83.82" y2="139.7" width="0.1524" layer="91"/>
+<wire x1="83.82" y1="139.7" x2="101.6" y2="139.7" width="0.1524" layer="91"/>
+<junction x="101.6" y="139.7"/>
+<pinref part="C10" gate="G$1" pin="2"/>
+<wire x1="71.12" y1="162.56" x2="71.12" y2="139.7" width="0.1524" layer="91"/>
+<wire x1="71.12" y1="139.7" x2="83.82" y2="139.7" width="0.1524" layer="91"/>
+<junction x="83.82" y="139.7"/>
+</segment>
+</net>
+<net name="N$12" class="0">
+<segment>
+<pinref part="R9" gate="G$1" pin="1"/>
+<wire x1="83.82" y1="167.64" x2="104.14" y2="167.64" width="0.1524" layer="91"/>
+<junction x="104.14" y="167.64"/>
+<pinref part="U4" gate="A" pin="PS/SYNC"/>
+<wire x1="104.14" y1="167.64" x2="106.68" y2="167.64" width="0.1524" layer="91"/>
+<pinref part="U4" gate="A" pin="EN"/>
+<pinref part="U4" gate="A" pin="VINA"/>
+<wire x1="104.14" y1="177.8" x2="106.68" y2="177.8" width="0.1524" layer="91"/>
+<wire x1="104.14" y1="177.8" x2="104.14" y2="172.72" width="0.1524" layer="91"/>
+<wire x1="104.14" y1="172.72" x2="106.68" y2="172.72" width="0.1524" layer="91"/>
+<wire x1="104.14" y1="172.72" x2="104.14" y2="167.64" width="0.1524" layer="91"/>
+<junction x="104.14" y="172.72"/>
+<pinref part="C11" gate="G$1" pin="1"/>
+<wire x1="83.82" y1="165.1" x2="83.82" y2="167.64" width="0.1524" layer="91"/>
+<junction x="83.82" y="167.64"/>
+</segment>
+</net>
+<net name="+3V3" class="0">
+<segment>
+<pinref part="U4" gate="A" pin="VOUT"/>
+<wire x1="142.24" y1="180.34" x2="144.78" y2="180.34" width="0.1524" layer="91"/>
+<label x="172.72" y="180.34" size="1.778" layer="95"/>
+<pinref part="C4" gate="G$1" pin="1"/>
+<wire x1="144.78" y1="180.34" x2="149.86" y2="180.34" width="0.1524" layer="91"/>
+<wire x1="149.86" y1="180.34" x2="162.56" y2="180.34" width="0.1524" layer="91"/>
+<wire x1="149.86" y1="172.72" x2="149.86" y2="180.34" width="0.1524" layer="91"/>
+<junction x="149.86" y="180.34"/>
+<pinref part="C9" gate="G$1" pin="1"/>
+<wire x1="162.56" y1="172.72" x2="162.56" y2="180.34" width="0.1524" layer="91"/>
+<junction x="162.56" y="180.34"/>
+<wire x1="162.56" y1="180.34" x2="170.18" y2="180.34" width="0.1524" layer="91"/>
+<pinref part="+3V1" gate="G$1" pin="+3V3"/>
+<wire x1="170.18" y1="180.34" x2="170.18" y2="182.88" width="0.1524" layer="91"/>
+<wire x1="142.24" y1="187.96" x2="144.78" y2="187.96" width="0.1524" layer="91"/>
+<wire x1="144.78" y1="187.96" x2="144.78" y2="180.34" width="0.1524" layer="91"/>
+<junction x="144.78" y="180.34"/>
+</segment>
+</net>
+<net name="N$9" class="0">
+<segment>
+<pinref part="U4" gate="A" pin="FB"/>
+<wire x1="106.68" y1="170.18" x2="101.6" y2="170.18" width="0.1524" layer="91"/>
+<wire x1="101.6" y1="170.18" x2="101.6" y2="187.96" width="0.1524" layer="91"/>
+<wire x1="101.6" y1="187.96" x2="142.24" y2="187.96" width="0.1524" layer="91"/>
+</segment>
+</net>

Commit message: Node 2 Power, i2 modiefied
Parts:
- added D1: ZPD, diode:ZPD
- added Q1: IRF9530, transistor-power:IRF9530
- added R10: 100k, rcl:R-EU_R0805
Connections:
- removed net 0V: C10.2, C11.2, C4.2, C9.2, U4.GND, U4.PGND
- removed net INT: R3.1, R8.1
- removed net N$8: C10.1, R9.2, U4.VIN
- removed net VCC: C5.1, C6.1, C7.1, C8.1
- new net +5V: C10.1, D1.C, Q1.D, R9.2, U4.VIN
- new net GNDA: R10.1, U4.PGND, U4.POWER_PAD
- new net INT_LI: R3.1
- new net INT_RTC: R8.1
- new net N$14: D1.A, Q1.G, R10.2
- new net N$15: G1.-, G2.-, G3.-
- net +3V3: now also C5.1, C6.1, C7.1, C8.1, U4.FB
- net GND: now also C10.2, C11.2, C4.2, C9.2, U4.GND
- net N$9: now also G1.+, G2.+, G3.+; no longer U4.FB
Other:
- moved on the sheet: C4, C9, G1, G2, G3, J1, LS1

Commit message: node2 modified
Parts:
- added U$1: MF-SMDF050, fuse:MF-SMDF050
Connections:
- new net N$8: D1.C, Q1.D, U$1.1
- net +5V: now also U$1.2; no longer D1.C, Q1.D
Changed lines of the file:
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@@
 <part name="P+2" library="supply1" deviceset="+5V" device=""/>
 <part name="GND5" library="supply1" deviceset="GND" device=""/>
+<part name="U$1" library="fuse" deviceset="MF-SMDF" device="" technology="050"/>
 </parts>
 <sheets>
@@
 <instance part="R10" gate="G$1" x="35.56" y="154.94" rot="R90"/>
 <instance part="GND6" gate="1" x="35.56" y="142.24"/>
-<instance part="P+2" gate="1" x="40.64" y="185.42"/>
+<instance part="P+2" gate="1" x="40.64" y="190.5"/>
 <instance part="GND5" gate="1" x="144.78" y="10.16"/>
+<instance part="U$1" gate="A" x="40.64" y="180.34" rot="R90"/>
 </instances>
 <busses>
@@
 </segment>
 <segment>
-<pinref part="Q1" gate="G$1" pin="D"/>
-<pinref part="D1" gate="G$1" pin="C"/>
-<wire x1="38.1" y1="172.72" x2="40.64" y2="172.72" width="0.1524" layer="91"/>
-<wire x1="40.64" y1="172.72" x2="40.64" y2="170.18" width="0.1524" layer="91"/>
+<pinref part="U$1" gate="A" pin="2"/>
 <pinref part="P+2" gate="1" pin="+5V"/>
-<wire x1="40.64" y1="172.72" x2="40.64" y2="182.88" width="0.1524" layer="91"/>
-<junction x="40.64" y="172.72"/>
+<wire x1="40.64" y1="185.42" x2="40.64" y2="187.96" width="0.1524" layer="91"/>
 </segment>
 </net>
@@
 </segment>
 </net>
+<net name="N$8" class="0">
+<segment>
+<pinref part="Q1" gate="G$1" pin="D"/>
+<pinref part="D1" gate="G$1" pin="C"/>
+<wire x1="38.1" y1="172.72" x2="40.64" y2="172.72" width="0.1524" layer="91"/>
+<wire x1="40.64" y1="172.72" x2="40.64" y2="170.18" width="0.1524" layer="91"/>
+<pinref part="U$1" gate="A" pin="1"/>
+<wire x1="40.64" y1="175.26" x2="40.64" y2="172.72" width="0.1524" layer="91"/>
+<junction x="40.64" y="172.72"/>
+</segment>
+</net>

Commit message: node 2 display
Parts:
- removed LS1: CMS-181325-078S, BlueHome:CMS-181325-078S
- added !!!MBR0530!!!, !!!MBR0530!!!1, !!!MBR0530!!!2: PD3S160, diode:PD3S160
- added !!!SI1308EDL!!!: (no value), zetex:NMOSSOT23
- added C12, C14: 1u, rcl:C-EUC0805
- added C13, C15: 100n, rcl:C-EUC0805
- added C16, C17: 100nF, rcl:C-EUC0805
- added C18: 1nF_5%, rcl:C-EUC0805
- added C19: 0.1µF, rcl:C-EUC0805
- added C20, C21, C22, C23, C28, C30, C33: 1µF, rcl:C-EUC0805
- added C24, C25, C27, C29, C31: 10µF, rcl:C-EUC0805
- added C26: 4.7µF, rcl:C-EUC0805
- added C32: 2.2µF, rcl:C-EUC0805
- added HM1: HDC2080DMBR, BlueHome:HDC2080DMBR
- added L2: 10µH, rcl:L-EUL1812
- added MK1: ICS-40180, BlueHome:ICS-40180
- added R11, R12, R13, R14: 10k, rcl:R-EU_R0805
- added R15: 470m, rcl:R-EU_R0805
- added U$2: SX8635, BlueHome:SX8635
Connections:
- net INT_LI renamed INT_TSL
- new net ADC: C32.2
- new net BS: J1.8
- new net BUSY_N: J1.9
- new net CSB: J1.12
- new net DC: J1.11
- new net GDR: !!!SI1308EDL!!!.G, J1.2
- new net INT_HDC: HM1.DRDY/INT
- new net N$13: HM1.SDA, R11.2
- new net N$16: R13.2, U$2.SCL
- new net N$17: R14.2, U$2.SDA
- new net N$18: C16.2, U$2.VDIG
- new net N$19: C17.2, U$2.VANA
- new net N$20: C18.2, U$2.CP
- new net N$21: C18.1, U$2.CN
- new net N$22: C32.1, MK1.OUTPUT
- new net N$23: !!!MBR0530!!!.A, !!!SI1308EDL!!!.D, C26.1, L2.2
- new net N$24: !!!MBR0530!!!1.A, !!!MBR0530!!!2.C, C26.2
- new net N$26: C31.2, C33.2, MK1.VDD
- new net RESE: !!!SI1308EDL!!!.S, J1.3, R15.2
- new net RESET: U$2.RESETB
- new net RST_N: J1.10
- new net SCL*: J1.13
- new net SDA*: J1.14
- new net TSCL: J1.6
- new net TSDA: J1.7
- new net VCOM: C19.2, J1.24
- new net VDD_18V: C20.2, J1.18
- new net VGH: !!!MBR0530!!!.C, C27.2, C30.2, J1.21
- new net VGL: !!!MBR0530!!!2.A, C28.2, C29.2, J1.23
- new net VOTP: C23.1, J1.19
- new net VSH: C21.2, J1.20
- new net VSHR: C22.2, J1.22
- new net VSL: J1.5
- new net VSLR: J1.4
- new net VSS: C19.1, C20.1, C21.1, C22.1, C23.2, J1.17
- net +3V3: now also C12.1, C13.1, C14.1, C15.1, C16.1, C17.1, C24.1, C25.1, C31.1, C33.1, HM1.VDD, IC1.VDD, J1.15, J1.16, L2.1, U$2.VDD
- net GND: now also !!!MBR0530!!!1.C, C12.2, C13.2, C14.2, C15.2, C24.2, C25.2, C27.1, C28.1, C29.1, C30.1, HM1.GND, MK1.GND, R15.1, U$2.GND_0, U$2.GND_1, U$2.GND_2, U$2.GND_3
- net INT_RTC: now also R8.2; no longer R8.1
- net N$4: now also R8.1; no longer R8.2
- net N$6: now also HM1.SCL, R12.2; no longer IC1.VDD
- net SCL: now also R12.1, R13.1
- net SDA: now also R11.1, R14.1
Other:
- moved on the sheet: C1, C2, C3, C5, C6, C7, C8, J1, R1, R2, R3, R5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

Commit message: restored
Parts:
- removed !!!MBR0530!!!, !!!MBR0530!!!1, !!!MBR0530!!!2: PD3S160, diode:PD3S160
- removed !!!SI1308EDL!!!: (no value), zetex:NMOSSOT23
- added D5, D6, D7: MBR0530, BlueHome:MBR0530
- added Q2: SI1308EDL-T1-GE3, BlueHome:SI1308EDL-T1-GE3
- added R16: 10k, rcl:R-EU_R0805
- C26: value 4.7µF -> 0.1µF
- L2: value 10µH -> 68µH
Connections:
- net GDR: now also Q2.G, R16.2; no longer !!!SI1308EDL!!!.G
- net GND: now also D5.K, R16.1; no longer !!!MBR0530!!!1.C
- net N$23: now also D6.A, Q2.D; no longer !!!MBR0530!!!.A, !!!SI1308EDL!!!.D
- net N$24: now also D5.A, D7.K; no longer !!!MBR0530!!!1.A, !!!MBR0530!!!2.C
- net N$8: now also Q1.S; no longer Q1.D
- net N$9: now also Q1.D
- net RESE: now also Q2.S; no longer !!!SI1308EDL!!!.S
- net VGH: now also D6.K; no longer !!!MBR0530!!!.C
- net VGL: now also D7.A; no longer !!!MBR0530!!!2.A
Other:
- moved on the sheet: Q1
