File: Node#2/Node#2.sch (EAGLE design)
At the start: 68 parts, among them IC1 TSL25911FN, J1 68712414522, Q1 IRF9530, Q2 SI1308EDL-T1-GE3, U2 RV8564C3, U4 TPS63001DRCT

Commit message: bi-colour_leds
Parts:
- added LED1, LED2, LED3, LED4, LED5, LED6: 156125YV73000, BlueHome:156125YV73000
Connections:
- new net LED0: LED1.K_1, LED2.K_1, LED3.K_1, LED4.K_1, LED5.K_1, LED6.K_1, U$2.GPIO0
- new net LED1: LED1.K_2, U$2.GPIO1
- new net LED2: LED2.K_2, U$2.GPIO2
- new net LED3: LED3.K_2, U$2.GPIO3
- new net LED4: LED4.K_2, U$2.GPIO4
- new net LED5: LED5.K_2, U$2.GPIO5
- new net LED6: LED6.K_2
- new net N$25: LED1.A_1, LED1.A_2, LED2.A_1, LED2.A_2
- new net N$27: LED3.A_1, LED3.A_2, LED4.A_1, LED4.A_2
- new net N$30: LED5.A_1, LED5.A_2, LED6.A_1, LED6.A_2
- new net N$34: U$2.GPIO6
- new net N$35: U$2.GPIO7
Changed lines of the file:
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@@
 <part name="D6" library="BlueHome" deviceset="MBR0530" device=""/>
 <part name="D7" library="BlueHome" deviceset="MBR0530" device=""/>
+<part name="LED1" library="BlueHome" deviceset="156125YV73000" device=""/>
+<part name="LED2" library="BlueHome" deviceset="156125YV73000" device=""/>
+<part name="LED3" library="BlueHome" deviceset="156125YV73000" device=""/>
+<part name="LED4" library="BlueHome" deviceset="156125YV73000" device=""/>
+<part name="LED5" library="BlueHome" deviceset="156125YV73000" device=""/>
+<part name="LED6" library="BlueHome" deviceset="156125YV73000" device=""/>
 </parts>
 <sheets>
@@
 <instance part="D6" gate="G$1" x="-210.82" y="78.74" rot="R90"/>
 <instance part="D7" gate="G$1" x="-180.34" y="93.98" rot="R270"/>
+<instance part="LED1" gate="G$1" x="218.44" y="-71.12"/>
+<instance part="LED2" gate="G$1" x="236.22" y="-78.74"/>
+<instance part="LED3" gate="G$1" x="218.44" y="-86.36"/>
+<instance part="LED4" gate="G$1" x="236.22" y="-93.98"/>
+<instance part="LED5" gate="G$1" x="218.44" y="-101.6"/>
+<instance part="LED6" gate="G$1" x="236.22" y="-109.22"/>
 </instances>
 <busses>
@@
 </segment>
 </net>
+<net name="N$25" class="0">
+<segment>
+<pinref part="LED2" gate="G$1" pin="A_1"/>
+<wire x1="264.16" y1="-73.66" x2="264.16" y2="-78.74" width="0.1524" layer="91"/>
+<wire x1="264.16" y1="-78.74" x2="261.62" y2="-78.74" width="0.1524" layer="91"/>
+<wire x1="264.16" y1="-78.74" x2="264.16" y2="-81.28" width="0.1524" layer="91"/>
+<junction x="264.16" y="-78.74"/>
+<pinref part="LED2" gate="G$1" pin="A_2"/>
+<wire x1="264.16" y1="-81.28" x2="261.62" y2="-81.28" width="0.1524" layer="91"/>
+<pinref part="LED1" gate="G$1" pin="A_2"/>
+<wire x1="243.84" y1="-73.66" x2="246.38" y2="-73.66" width="0.1524" layer="91"/>
+<pinref part="LED1" gate="G$1" pin="A_1"/>
+<wire x1="246.38" y1="-73.66" x2="264.16" y2="-73.66" width="0.1524" layer="91"/>
+<wire x1="243.84" y1="-71.12" x2="246.38" y2="-71.12" width="0.1524" layer="91"/>
+<wire x1="246.38" y1="-71.12" x2="246.38" y2="-73.66" width="0.1524" layer="91"/>
+<junction x="246.38" y="-73.66"/>
+</segment>
+</net>
+<net name="LED0" class="0">
+<segment>
+<pinref part="U$2" gate="G$1" pin="GPIO0"/>
+<wire x1="193.04" y1="-71.12" x2="198.12" y2="-71.12" width="0.1524" layer="91"/>
+<label x="193.04" y="-71.12" size="1.778" layer="95"/>
+</segment>
+<segment>
+<pinref part="LED1" gate="G$1" pin="K_1"/>
+<wire x1="218.44" y1="-71.12" x2="213.36" y2="-71.12" width="0.1524" layer="91"/>
+<label x="213.36" y="-71.12" size="1.778" layer="95"/>
+</segment>
+<segment>
+<pinref part="LED2" gate="G$1" pin="K_1"/>
+<wire x1="236.22" y1="-78.74" x2="213.36" y2="-78.74" width="0.1524" layer="91"/>
+<label x="213.36" y="-78.74" size="1.778" layer="95"/>
+</segment>
+<segment>
+<pinref part="LED3" gate="G$1" pin="K_1"/>
+<wire x1="218.44" y1="-86.36" x2="213.36" y2="-86.36" width="0.1524" layer="91"/>
+<label x="213.36" y="-86.36" size="1.778" layer="95"/>
+</segment>
+<segment>
+<pinref part="LED4" gate="G$1" pin="K_1"/>
+<wire x1="236.22" y1="-93.98" x2="213.36" y2="-93.98" width="0.1524" layer="91"/>
+<label x="213.36" y="-93.98" size="1.778" layer="95"/>
+</segment>
+<segment>
+<pinref part="LED5" gate="G$1" pin="K_1"/>
+<wire x1="218.44" y1="-101.6" x2="213.36" y2="-101.6" width="0.1524" layer="91"/>
+<label x="213.36" y="-101.6" size="1.778" layer="95"/>
+</segment>
+<segment>
+<pinref part="LED6" gate="G$1" pin="K_1"/>
+<wire x1="236.22" y1="-109.22" x2="213.36" y2="-109.22" width="0.1524" layer="91"/>
+<label x="213.36" y="-109.22" size="1.778" layer="95"/>
+</segment>
+</net>
+<net name="LED1" class="0">
+<segment>
+<pinref part="U$2" gate="G$1" pin="GPIO1"/>
+<wire x1="193.04" y1="-73.66" x2="198.12" y2="-73.66" width="0.1524" layer="91"/>
+<label x="193.04" y="-73.66" size="1.778" layer="95"/>
+</segment>
+<segment>
+<pinref part="LED1" gate="G$1" pin="K_2"/>
+<wire x1="218.44" y1="-73.66" x2="213.36" y2="-73.66" width="0.1524" layer="91"/>
+<label x="213.36" y="-73.66" size="1.778" layer="95"/>
+</segment>
+</net>
+<net name="LED2" class="0">
+<segment>
+<pinref part="U$2" gate="G$1" pin="GPIO2"/>
+<wire x1="193.04" y1="-76.2" x2="198.12" y2="-76.2" width="0.1524" layer="91"/>
+<label x="193.04" y="-76.2" size="1.778" layer="95"/>
+</segment>
+<segment>
+<pinref part="LED2" gate="G$1" pin="K_2"/>
+<wire x1="236.22" y1="-81.28" x2="213.36" y2="-81.28" width="0.1524" layer="91"/>
+<label x="213.36" y="-81.28" size="1.778" layer="95"/>
+</segment>
+</net>
+<net name="LED3" class="0">
+<segment>
+<pinref part="U$2" gate="G$1" pin="GPIO3"/>
+<wire x1="193.04" y1="-78.74" x2="198.12" y2="-78.74" width="0.1524" layer="91"/>
+<label x="193.04" y="-78.74" size="1.778" layer="95"/>
+</segment>
+<segment>
+<pinref part="LED3" gate="G$1" pin="K_2"/>
+<wire x1="218.44" y1="-88.9" x2="213.36" y2="-88.9" width="0.1524" layer="91"/>
+<label x="213.36" y="-88.9" size="1.778" layer="95"/>
+</segment>
+</net>
+<net name="LED4" class="0">
+<segment>
+<pinref part="U$2" gate="G$1" pin="GPIO4"/>
+<wire x1="193.04" y1="-81.28" x2="198.12" y2="-81.28" width="0.1524" layer="91"/>
+<label x="193.04" y="-81.28" size="1.778" layer="95"/>
+</segment>
+<segment>
+<pinref part="LED4" gate="G$1" pin="K_2"/>
+<wire x1="236.22" y1="-96.52" x2="213.36" y2="-96.52" width="0.1524" layer="91"/>
+<label x="213.36" y="-96.52" size="1.778" layer="95"/>
+</segment>
+</net>
+<net name="LED5" class="0">
+<segment>
+<pinref part="U$2" gate="G$1" pin="GPIO5"/>
+<wire x1="193.04" y1="-83.82" x2="198.12" y2="-83.82" width="0.1524" layer="91"/>
+<label x="193.04" y="-83.82" size="1.778" layer="95"/>
+</segment>
+<segment>
+<pinref part="LED5" gate="G$1" pin="K_2"/>
+<wire x1="218.44" y1="-104.14" x2="213.36" y2="-104.14" width="0.1524" layer="91"/>
+<label x="213.36" y="-104.14" size="1.778" layer="95"/>
+</segment>
+</net>
+<net name="N$34" class="0">
+<segment>
+<pinref part="U$2" gate="G$1" pin="GPIO6"/>
+<wire x1="193.04" y1="-86.36" x2="198.12" y2="-86.36" width="0.1524" layer="91"/>
+</segment>
+</net>
+<net name="N$35" class="0">
+<segment>
+<pinref part="U$2" gate="G$1" pin="GPIO7"/>
+<wire x1="193.04" y1="-88.9" x2="198.12" y2="-88.9" width="0.1524" layer="91"/>
+</segment>
+</net>
+<net name="N$27" class="0">
+<segment>
+<pinref part="LED4" gate="G$1" pin="A_1"/>
+<wire x1="264.16" y1="-88.9" x2="264.16" y2="-93.98" width="0.1524" layer="91"/>
+<wire x1="264.16" y1="-93.98" x2="261.62" y2="-93.98" width="0.1524" layer="91"/>
+<wire x1="264.16" y1="-93.98" x2="264.16" y2="-96.52" width="0.1524" layer="91"/>
+<junction x="264.16" y="-93.98"/>
+<pinref part="LED4" gate="G$1" pin="A_2"/>
+<wire x1="264.16" y1="-96.52" x2="261.62" y2="-96.52" width="0.1524" layer="91"/>
+<pinref part="LED3" gate="G$1" pin="A_2"/>
+<wire x1="243.84" y1="-88.9" x2="246.38" y2="-88.9" width="0.1524" layer="91"/>
+<pinref part="LED3" gate="G$1" pin="A_1"/>
+<wire x1="246.38" y1="-88.9" x2="264.16" y2="-88.9" width="0.1524" layer="91"/>
+<wire x1="243.84" y1="-86.36" x2="246.38" y2="-86.36" width="0.1524" layer="91"/>
+<wire x1="246.38" y1="-86.36" x2="246.38" y2="-88.9" width="0.1524" layer="91"/>
+<junction x="246.38" y="-88.9"/>
+</segment>
+</net>
+<net name="N$30" class="0">
+<segment>
+<pinref part="LED6" gate="G$1" pin="A_1"/>
+<wire x1="264.16" y1="-104.14" x2="264.16" y2="-109.22" width="0.1524" layer="91"/>
+<wire x1="264.16" y1="-109.22" x2="261.62" y2="-109.22" width="0.1524" layer="91"/>
+<wire x1="264.16" y1="-109.22" x2="264.16" y2="-111.76" width="0.1524" layer="91"/>
+<junction x="264.16" y="-109.22"/>
+<pinref part="LED6" gate="G$1" pin="A_2"/>
+<wire x1="264.16" y1="-111.76" x2="261.62" y2="-111.76" width="0.1524" layer="91"/>
+<pinref part="LED5" gate="G$1" pin="A_2"/>
+<wire x1="243.84" y1="-104.14" x2="246.38" y2="-104.14" width="0.1524" layer="91"/>
+<pinref part="LED5" gate="G$1" pin="A_1"/>
+<wire x1="246.38" y1="-104.14" x2="264.16" y2="-104.14" width="0.1524" layer="91"/>
+<wire x1="243.84" y1="-101.6" x2="246.38" y2="-101.6" width="0.1524" layer="91"/>
+<wire x1="246.38" y1="-101.6" x2="246.38" y2="-104.14" width="0.1524" layer="91"/>
+<junction x="246.38" y="-104.14"/>
+</segment>
+</net>
+<net name="LED6" class="0">
+<segment>
+<pinref part="LED6" gate="G$1" pin="K_2"/>
+<wire x1="236.22" y1="-111.76" x2="213.36" y2="-111.76" width="0.1524" layer="91"/>
+<label x="213.36" y="-111.76" size="1.778" layer="95"/>
+</segment>
+</net>

Commit message: small changes
Parts:
- removed C1: (no value), rcl:C-EUC0805
- removed C2: 1u, rcl:C-EUC0805
- removed C3: 100n, rcl:C-EUC0805
- removed R11, R12, R13, R14, R2, R4, R6, R7: 10k, rcl:R-EU_R0805
- added R17: 1.5M, rcl:R-EU_R0805
- added R18: 10k, rcl:R-EU_R0805
- added U$3, U$4, U$5, U$6, U$7: TOUCH_BUTTON, BlueHome:TOUCH_BUTTON
- added U$8: WHEEL, BlueHome:WHEEL
- R1: value (none) -> 10k
- R3, R8: value 10k -> 4.7k
- R5: value 10k -> 1M
Connections:
- net ADC renamed ADC1
- net GNDA renamed V-
- removed net N$1: IC1.SDA, R4.2
- removed net N$13: HM1.SDA, R11.2
- removed net N$16: R13.2, U$2.SCL
- removed net N$17: R14.2, U$2.SDA
- removed net N$2: IC1.SCL, R2.2
- removed net N$25: LED1.A_1, LED1.A_2, LED2.A_1, LED2.A_2
- removed net N$27: LED3.A_1, LED3.A_2, LED4.A_1, LED4.A_2
- removed net N$3: IC1.INT, R3.2
- removed net N$30: LED5.A_1, LED5.A_2, LED6.A_1, LED6.A_2
- removed net N$4: R8.1, U2.INT
- removed net N$5: R7.2, U2.SCL
- removed net N$6: HM1.SCL, R12.2
- removed net N$7: R6.2, U2.SDA
- new net ADC2: R17.2, R5.1
- new net INT_SX: U$2.INTB
- new net N$28: U$2.CAP1, U$3.BUTTON
- new net N$29: U$2.CAP2, U$4.BUTTON
- new net N$31: U$2.CAP3, U$5.BUTTON
- new net N$32: U$2.CAP4, U$6.BUTTON
- new net N$33: U$2.CAP0, U$7.BUTTON
- new net SEG1: U$2.CAP5, U$8.SEG1
- new net SEG2: U$2.CAP6, U$8.SEG2
- new net SEG3: U$2.CAP7, U$8.SEG3
- new net SEG4: U$2.CAP8, U$8.SEG4
- new net V+: C10.1, R9.2, U4.VIN
- net +3V3: now also LED1.A_1, LED1.A_2, LED2.A_1, LED2.A_2, LED3.A_1, LED3.A_2, LED4.A_1, LED4.A_2, LED5.A_1, LED5.A_2, LED6.A_1, LED6.A_2, R1.2, R3.2, R8.2
- net +5V: now also R5.2; no longer C10.1, R9.2, U4.VIN
- net CSB: now also R1.1, R18.2
- net GND: now also HM1.ADDR, R17.1, R18.1, U2.CLKOE
- net INT_RTC: now also U2.INT; no longer R8.2
- net INT_TSL: now also IC1.INT; no longer R3.1
- net SCL: now also HM1.SCL, IC1.SCL, U$2.SCL, U2.SCL; no longer R12.1, R13.1, R2.1, R7.1
- net SDA: now also HM1.SDA, IC1.SDA, U$2.SDA, U2.SDA; no longer R11.1, R14.1, R4.1, R6.1
- net TSCL: now also R8.1
- net TSDA: now also R3.1
Other:
- moved on the sheet: C19, C20, C21, C22, C23, C24, C25, C26, C27, C28, C29, C30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

Commit message: node2 spi, rtc
Parts:
- removed Q1: IRF9530, transistor-power:IRF9530
- added !!!FDN304PZ!!!: BSS84, transistor-small-signal:BSS84
- added C1, C2: 1µF, rcl:C-EUC0805
- added C3: 100mF, rcl:C-EU050-055X075
- added D2: MUR150RL, diode:MUR150RL
- C26: value 0.1µF -> 4.7µF
- L1: device rcl:L-EUL1812 -> rcl:L-EUL4532P
- L2: value 68µH -> 10µH
Connections:
- net CSB renamed CS
- removed net SCL*: J1.13
- removed net SDA*: J1.14
- new net +3V3_RTC: C3.1, C7.2, C8.2, D2.C, U2.VDD
- new net MOSI: J1.14, R3.1
- new net SCLK: J1.13, R8.1
- net +3V3: now also D2.A; no longer C7.1, C8.1
- net GND: now also C1.1, C2.2, C3.2, C7.1, C8.1; no longer C7.2, C8.2
- net N$14: now also !!!FDN304PZ!!!.G; no longer Q1.G
- net N$8: now also !!!FDN304PZ!!!.S; no longer Q1.S
- net N$9: now also !!!FDN304PZ!!!.D; no longer Q1.D
- net SDA: no longer U2.VDD
- net TSCL: no longer R8.1
- net TSDA: no longer R3.1
- net VSL: now also C1.2
- net VSLR: now also C2.1
Other:
- note added: "3-/4-wire"
- note added: "Negative Gate Voltage"
- note added: "Positive Gate Voltage"
- note added: "VDD"
- note added: "VDDIO"
- moved on the sheet: C7, C8, D1, G1, G2, G3, R1, R10, R18, R3, R8, U$1
